File: EngineController.kicad_sch (KiCad schematic)
At the start: 37 parts, among them J1 RBUS, U1 ESP32-S3, Y1 R940000171

Commit message: Schematic done, components layed out, sensors wired up
Connections:
- net BUCK_EN: no longer U1.18 (GPIO13/ADC2_CH2)
- net HSPI_MISO: now also U1.39 (GPIO34); no longer U1.40 (GPIO35)
- net HSPI_MOSI: now also U1.40 (GPIO35); no longer U1.38 (GPIO33)
- net HSPI_SCLK: now also U1.38 (GPIO33); no longer U1.39 (GPIO34)
- net VSPI_MISO: now also U1.32 (SPICS0/GPIO29); no longer U1.33 (SPICLK/GPIO30)
- net VSPI_MOSI: now also U1.33 (SPICLK/GPIO30); no longer U1.31 (SPIWP/GPIO28)
- net VSPI_SCLK: now also U1.31 (SPIWP/GPIO28); no longer U1.32 (SPICS0/GPIO29)
- net BUCKP_EN: now reaches U1.19 (GPIO14/ADC2_CH3)
- new net BUCKC_EN: U1.18 (GPIO13/ADC2_CH2)
- no-connect marks 17 -> 16
Changed lines of the file:
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@@
   (junction (at 135.89 143.51) (diameter 0) (color 0 0 0 0)
   )
-  (no_connect (at 69.85 105.41))
   (no_connect (at 135.89 115.57))
   (no_connect (at 135.89 105.41))
@@
     (stroke (width 0) (type default))
   )
-  (wire (pts (xy 205.994 123.19) (xy 214.884 123.19))
-    (stroke (width 0) (type default))
-  )
   (wire (pts (xy 58.42 21.59) (xy 58.42 26.67))
     (stroke (width 0) (type default))
@@
     (effects (font (size 1.27 1.27)) (justify left bottom))
   )
-  (label "MOSI" (at 220.98 81.28 0) (fields_autoplaced)
+  (label "BUCKP_EN" (at 69.85 105.41 180) (fields_autoplaced)
+    (effects (font (size 1.27 1.27)) (justify right bottom))
+  )
+  (label "HSPI_MOSI" (at 220.98 81.28 0) (fields_autoplaced)
     (effects (font (size 1.27 1.27)) (justify left bottom))
   )
@@
     (effects (font (size 1.27 1.27)) (justify left bottom))
   )
-  (label "MISO" (at 220.98 83.82 0) (fields_autoplaced)
-    (effects (font (size 1.27 1.27)) (justify left bottom))
-  )
-  (label "SCLK" (at 220.98 78.74 0) (fields_autoplaced)
+  (label "HSPI_MISO" (at 220.98 83.82 0) (fields_autoplaced)
+    (effects (font (size 1.27 1.27)) (justify left bottom))
+  )
+  (label "HSPI_SCLK" (at 220.98 78.74 0) (fields_autoplaced)
     (effects (font (size 1.27 1.27)) (justify left bottom))
   )
@@
     (effects (font (size 1.27 1.27)) (justify right bottom))
   )
-  (label "VSPI_SCLK" (at 135.89 85.09 0) (fields_autoplaced)
+  (label "VSPI_SCLK" (at 135.89 82.55 0) (fields_autoplaced)
     (effects (font (size 1.27 1.27)) (justify left bottom))
   )
@@
     (effects (font (size 1.27 1.27)) (justify right bottom))
   )
-  (label "HSPI_SCLK" (at 135.89 97.79 0) (fields_autoplaced)
+  (label "HSPI_SCLK" (at 135.89 95.25 0) (fields_autoplaced)
     (effects (font (size 1.27 1.27)) (justify left bottom))
   )
@@
     (effects (font (size 1.27 1.27)) (justify left bottom))
   )
-  (label "VSPI_MISO" (at 135.89 87.63 0) (fields_autoplaced)
+  (label "VSPI_MISO" (at 135.89 85.09 0) (fields_autoplaced)
     (effects (font (size 1.27 1.27)) (justify left bottom))
   )
@@
     (effects (font (size 1.27 1.27)) (justify left bottom))
   )
-  (label "PyroPWR" (at 205.994 123.19 0) (fields_autoplaced)
-    (effects (font (size 1.27 1.27)) (justify left bottom))
-  )
-  (label "BUCK_EN" (at 69.85 102.87 180) (fields_autoplaced)
+  (label "BUCKC_EN" (at 69.85 102.87 180) (fields_autoplaced)
     (effects (font (size 1.27 1.27)) (justify right bottom))
   )
@@
     (effects (font (size 1.27 1.27)) (justify left bottom))
   )
-  (label "VSPI_MOSI" (at 135.89 82.55 0) (fields_autoplaced)
+  (label "VSPI_MOSI" (at 135.89 87.63 0) (fields_autoplaced)
     (effects (font (size 1.27 1.27)) (justify left bottom))
   )
@@
     (effects (font (size 1.27 1.27)) (justify left bottom))
   )
-  (label "HSPI_MISO" (at 135.89 100.33 0) (fields_autoplaced)
+  (label "HSPI_MISO" (at 135.89 97.79 0) (fields_autoplaced)
     (effects (font (size 1.27 1.27)) (justify left bottom))
   )
@@
     (effects (font (size 1.27 1.27)) (justify right bottom))
   )
-  (label "HSPI_MOSI" (at 135.89 95.25 0) (fields_autoplaced)
+  (label "HSPI_MOSI" (at 135.89 100.33 0) (fields_autoplaced)
     (effects (font (size 1.27 1.27)) (justify left bottom))
   )
@@
     )
   )
-  (hierarchical_label "PyroPWR" (shape output) (at 214.884 123.19 0) (fields_autoplaced)
-    (effects (font (size 1.27 1.27)) (justify left))
-  )
   (hierarchical_label "Cont 1" (shape input) (at 214.884 130.556 0) (fields_autoplaced)

Commit message: Wired up more stuff
Connections:
- net VSPI_MISO: now also U1.31 (SPIWP/GPIO28); no longer U1.32 (SPICS0/GPIO29)
- net VSPI_SCLK: now also U1.32 (SPICS0/GPIO29); no longer U1.31 (SPIWP/GPIO28)
Changed lines of the file:
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@@
+    (stroke (width 0) (type default))
+  )
+  (wire (pts (xy 214.884 123.952) (xy 207.264 123.952))
     (stroke (width 0) (type default))
   )
@@
     (effects (font (size 1.27 1.27)) (justify left bottom))
   )
+  (label "BUCKP_EN" (at 207.264 123.952 180) (fields_autoplaced)
+    (effects (font (size 1.27 1.27)) (justify right bottom))
+  )
+  (label "BUCKC_EN" (at 226.06 21.59 180) (fields_autoplaced)
+    (effects (font (size 1.27 1.27)) (justify right bottom))
+  )
   (label "CHIP_PU" (at 36.83 165.1 180) (fields_autoplaced)
     (effects (font (size 1.27 1.27)) (justify right bottom))
@@
     (effects (font (size 1.27 1.27)) (justify right bottom))
   )
-  (label "VSPI_SCLK" (at 135.89 82.55 0) (fields_autoplaced)
+  (label "VSPI_SCLK" (at 135.89 85.09 0) (fields_autoplaced)
     (effects (font (size 1.27 1.27)) (justify left bottom))
   )
@@
     (effects (font (size 1.27 1.27)) (justify left bottom))
   )
-  (label "VSPI_MISO" (at 135.89 85.09 0) (fields_autoplaced)
+  (label "VSPI_MISO" (at 135.89 82.55 0) (fields_autoplaced)
     (effects (font (size 1.27 1.27)) (justify left bottom))
   )
@@
   )
   (label "CAN_RX" (at 69.85 72.39 180) (fields_autoplaced)
-    (effects (font (size 1.27 1.27)) (justify right bottom))
-  )
-  (label "BUCK_EN" (at 226.06 21.59 180) (fields_autoplaced)
     (effects (font (size 1.27 1.27)) (justify right bottom))
   )
@@
     )
   )
+  (hierarchical_label "BUCKP_EN" (shape output) (at 214.884 123.952 0) (fields_autoplaced)
+    (effects (font (size 1.27 1.27)) (justify left))
+  )
   (hierarchical_label "Cont 1" (shape input) (at 214.884 130.556 0) (fields_autoplaced)
