File: pressure_sensor_sch.kicad_sch (KiCad schematic)
At the start: 53 parts, among them J13 1053131104, U8 ADS131M06IPBS

Commit message: v1.2
Connections:
- net AIN0N: now also C73.2, J13.3, JP31.2 (B), R61.2; no longer C73.2, J13.3, JP31.2 (B), R61.2
- net AIN0P: now also C73.1, R61.1, R61.2, R61.2; no longer C73.1, R61.1, R61.2, R61.2
- net AIN1N: now also C73.2, J13.3, JP31.2 (B), R61.2; no longer C73.2, J13.3, JP31.2 (B), R61.2
- net AIN1P: now also C73.1, R61.1, R61.2, R61.2; no longer C73.1, R61.1, R61.2, R61.2
- net AIN2N: now also C73.2, J13.3, JP31.2 (B), R61.2; no longer C73.2, J13.3, JP31.2 (B), R61.2
- net AIN2P: now also C73.1, R61.1, R61.2, R61.2; no longer C73.1, R61.1, R61.2, R61.2
- net AIN3N: now also C73.2, J13.3, JP31.2 (B), R61.2; no longer C73.2, J13.3, JP31.2 (B), R61.2
- net AIN3P: now also C73.1, R61.1, R61.2, R61.2; no longer C73.1, R61.1, R61.2, R61.2
- net AIN4N: now also C73.2, J13.3, JP31.2 (B), R61.2; no longer C73.2, J13.3, JP31.2 (B), R61.2
- net AIN4P: now also C73.1, R61.1, R61.2, R61.2; no longer C73.1, R61.1, R61.2, R61.2
- net AIN5N: now also C73.2, J13.3, JP31.2 (B), R61.2; no longer C73.2, J13.3, JP31.2 (B), R61.2
- net AIN5P: now also C73.1, R61.1, R61.2, R61.2; no longer C73.1, R61.1, R61.2, R61.2

Commit message: More Based
Parts:
- added C39: 220nF, Capacitor_SMD:C_0402_1005Metric, symbol Device:C_Small
- renumbered U8 to U7
Connections:
- net GND: now also U7.28 (AGND), C39.2; no longer J13.4, JP31.1 (A)
- net at U7.24 (CAP): now also C39.1
- new net GNDA: J13.4, JP31.1 (A)
- no-connect marks 1 -> 3
