File: pressure_sensor_sch.kicad_sch (KiCad schematic)
At the start: 83 parts, among them J10 1053131104, J11 1053131104, J13 1053131104, J6 1053131104, J8 1053131104, J9 1053131104, U7 ADS131M06IPBS

Commit message: review 3 changes
Connections:
- net DRDY: now reaches U7.18 (DRDY)
- no-connect marks 2 -> 1
Changed lines of the file:
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@@
 	)
 	(no_connect
-		(at 98.298 116.84)
-	)
-	(no_connect
 		(at 32.258 114.3)
 	)
@@
 		)
 	)
+	(hierarchical_label "DRDY"
+		(shape bidirectional)
+		(at 98.298 116.84 0)
+		(fields_autoplaced yes)
+		(effects
+			(font
+				(size 1.27 1.27)
+			)
+			(justify left)
+		)
+	)
 	(hierarchical_label "ADS_SCLK"
 		(shape bidirectional)
@@
 			)
 		)
-		(property "Datasheet" "ADS131M06IPBS"
+		(property "Datasheet" "https://www.ti.com/lit/ds/symlink/ads131m06.pdf?ts=1722711447211&ref_url=https%253A%252F%252Fwww.ti.com%252Fproduct%252FADS131M06%253Fbm-verify%253DAAQAAAAJ_____3PRcak1s9y645AuuHNjtl9rOtrOIaOoIVylsudph4b42jws10PfoUc0NN8_vn4A5W1PRfakw0bMSz4jfLGW4zaYkLbaDcvq5L5_zHo15yGpMW7BVF3od7cx9KhugtbVdriNFDBo5LRJV0MvT1XGnlQPXQsUQtS6SiiLh9zAg47OOFflajmXwhRg6KqjRqyBOY1aoAJpzpQG_9El4vVs_b69ddXI-wn4pOsqD4OqvW4Iuar98OBh1F0vSQESnFJRUPIJBo_njnga3v0Ss-YlF-leunJX_IX177A5irbWwsOW0wVB"
 			(at 32.258 81.28 0)
 			(effects
