File: Ricardo-Stark.kicad_pcb (KiCad board)
At the start: 4 copper layers, 105 x 50 mm, 256 parts, among them IC1 TPS61089RNRR, IC2 AP2205-W5-7, IC3 AP2205-W5-7, IC4 TPS61089RNRR, J1 RBUS, J10 1053131104, J11 1053131104, J12 Conn_01x02_Male, J13 Micro_SD_Card_Det, J2 USB_C_Receptacle_USB2.0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

Commit message: Last commit wasnt based enough, forgot analogue ground isolation
Parts:
- moved R35 0.45 mm to (111.9, 96.5)
Routing:
- net GND: track 68.4 -> 75.4 mm, vias 138 -> 141
- net +12V: vias 11 -> 10
