File: Ricardo-Stark.kicad_pcb (KiCad board)
At the start: 4 copper layers, 259 parts, among them IC1 TPS61089RNRR, IC2 AP2205-W5-7, IC3 AP2205-W5-7, IC4 TPS61089RNRR, J1 RBUS, J10 1053131104, J11 1053131104, J12 Conn_01x02_Male, J13 Micro_SD_Card_Det, J2 USB_C_Receptacle_USB2.0, J3 ServoCH1, J4 ServoCH2, J5 GPIO Breakout, J6 1053131104, J7 1053131104, J8 1053131104, J9 1053131104, Q2 BUK9M11-40EX, U1 ESP32-S3, U10 SiC437BED-T1-GE3, U2 SN65HVD230, U3 LM66200DRLR, U4 MAX77827AEFD+T, U5 SC4215, U6 SiC437BED-T1-GE3, U7 ADS131M06IPBS, U8 TPS259621DDAT, U9 859-LTV-247, Y1 R940000171

Commit message: Sized sensor resistors and more routing
Parts:
- removed C38, C43, C44, C45, C46, C47: 10nF, Capacitor_SMD:C_0402_1005Metric
- removed C71: 2.2nF, Capacitor_SMD:C_0402_1005Metric
- removed C72: 1uF, Capacitor_SMD:C_0603_1608Metric
- removed C79: 1uF, Capacitor_SMD:C_0402_1005Metric
- removed J10, J11, J6, J8, J9: 1053131104, Connector_Molex:Molex_Nano-Fit_105313-xx04_1x04_P2.50mm_Horizontal
- removed JP11, JP13, JP14, JP15, JP17, JP19, JP2, JP4, JP6, JP7: SolderJumper_3_Open, Jumper:SolderJumper-3_P1.3mm_Open_RoundedPad1.0x1.5mm_NumberLabels
- removed JP12, JP16, JP18, JP3, JP9: SolderJumper_2_Open, Jumper:SolderJumper-2_P1.3mm_Open_RoundedPad1.0x1.5mm
- removed R42, R46, R47, R54, R55: 90k, Resistor_SMD:R_0402_1005Metric
- removed R43, R49, R50, R56, R57: 31.7k, Resistor_SMD:R_0402_1005Metric
- removed R44, R52, R53, R58, R59: 10k, Resistor_SMD:R_0402_1005Metric
- removed U8: TPS259621DDAT, EFuse:SO-PP-DDA-8_TEX
- added C86: 100nF, Capacitor_SMD:C_0402_1005Metric, F.Cu at (205.1, 69.6)
- added C87: 2.2nF, Capacitor_SMD:C_0402_1005Metric, F.Cu at (207.9, 74.2)
- added C88: 1uF, Capacitor_SMD:C_0603_1608Metric, F.Cu at (201.2, 69.3)
- added J14: 1053131104, Connector_Molex:Molex_Nano-Fit_105313-xx04_1x04_P2.50mm_Horizontal, F.Cu at (127.6, 69.3)
- added J15: 1053131104, Connector_Molex:Molex_Nano-Fit_105313-xx04_1x04_P2.50mm_Horizontal, F.Cu at (123.2, 90.2)
- added J16: 1053131104, Connector_Molex:Molex_Nano-Fit_105313-xx04_1x04_P2.50mm_Horizontal, F.Cu at (135.4, 95.2)
- added J17: 1053131104, Connector_Molex:Molex_Nano-Fit_105313-xx04_1x04_P2.50mm_Horizontal, F.Cu at (150.1, 95.2)
- added J18: 1053131104, Connector_Molex:Molex_Nano-Fit_105313-xx04_1x04_P2.50mm_Horizontal, F.Cu at (166.1, 95.2)
- added JP20: SolderJumper_3_Open, Jumper:SolderJumper-3_P1.3mm_Open_RoundedPad1.0x1.5mm_NumberLabels, F.Cu at (143.2, 75.2)
- added JP21: SolderJumper_3_Open, Jumper:SolderJumper-3_P1.3mm_Open_RoundedPad1.0x1.5mm_NumberLabels, F.Cu at (127.3, 72.7)
- added JP22: SolderJumper_3_Open, Jumper:SolderJumper-3_P1.3mm_Open_RoundedPad1.0x1.5mm_NumberLabels, F.Cu at (127.3, 75.3)
- added JP23: SolderJumper_2_Open, iclr:SmallerSolderJP, F.Cu at (132.9, 72.0)
- added JP24: SolderJumper_3_Open, Jumper:SolderJumper-3_P1.3mm_Open_RoundedPad1.0x1.5mm_NumberLabels, F.Cu at (123.5, 65.6)
- added JP25: SolderJumper_3_Open, Jumper:SolderJumper-3_P1.3mm_Open_RoundedPad1.0x1.5mm_NumberLabels, F.Cu at (-90.8, 61.4)
- added JP26: SolderJumper_3_Open, Jumper:SolderJumper-3_P1.3mm_Open_RoundedPad1.0x1.5mm_NumberLabels, F.Cu at (-85.2, 40.1)
- added JP27: SolderJumper_2_Open, iclr:SmallerSolderJP, F.Cu at (-91.7, 69.5)
- added JP28: SolderJumper_3_Open, Jumper:SolderJumper-3_P1.3mm_Open_RoundedPad1.0x1.5mm_NumberLabels, F.Cu at (-85.2, 43.7)
- added JP29: SolderJumper_3_Open, Jumper:SolderJumper-3_P1.3mm_Open_RoundedPad1.0x1.5mm_NumberLabels, F.Cu at (-85.2, 47.2)
- added JP30: SolderJumper_3_Open, Jumper:SolderJumper-3_P1.3mm_Open_RoundedPad1.0x1.5mm_NumberLabels, F.Cu at (-85.2, 50.8)
- added JP31: SolderJumper_2_Open, iclr:SmallerSolderJP, F.Cu at (-91.7, 72.0)
- added JP32: SolderJumper_3_Open, Jumper:SolderJumper-3_P1.3mm_Open_RoundedPad1.0x1.5mm_NumberLabels, F.Cu at (-85.2, 54.3)
- added JP33: SolderJumper_3_Open, Jumper:SolderJumper-3_P1.3mm_Open_RoundedPad1.0x1.5mm_NumberLabels, F.Cu at (-85.2, 57.9)
- added JP34: SolderJumper_3_Open, Jumper:SolderJumper-3_P1.3mm_Open_RoundedPad1.0x1.5mm_NumberLabels, F.Cu at (-85.2, 61.4)
- added JP35: SolderJumper_2_Open, iclr:SmallerSolderJP, F.Cu at (-91.7, 74.5)
- added JP36: SolderJumper_3_Open, Jumper:SolderJumper-3_P1.3mm_Open_RoundedPad1.0x1.5mm_NumberLabels, F.Cu at (-79.5, 40.1)
- added JP37: SolderJumper_3_Open, Jumper:SolderJumper-3_P1.3mm_Open_RoundedPad1.0x1.5mm_NumberLabels, F.Cu at (-79.5, 43.7)
- added JP38: SolderJumper_3_Open, Jumper:SolderJumper-3_P1.3mm_Open_RoundedPad1.0x1.5mm_NumberLabels, F.Cu at (-79.5, 47.2)
- added JP39: SolderJumper_2_Open, iclr:SmallerSolderJP, F.Cu at (-91.7, 77.0)
- added JP40: SolderJumper_3_Open, Jumper:SolderJumper-3_P1.3mm_Open_RoundedPad1.0x1.5mm_NumberLabels, F.Cu at (-79.5, 50.8)
- added R100: 10k, Resistor_SMD:R_0402_1005Metric, F.Cu at (-85.8, 76.1)
- added R101: 31.6k, Resistor_SMD:R_0402_1005Metric, F.Cu at (-82.9, 64.2)
- added R102: 49, Resistor_SMD:R_0402_1005Metric, F.Cu at (-82.9, 66.2)
- added R103: 58.4k, Resistor_SMD:R_0402_1005Metric, F.Cu at (-82.9, 68.2)
- added R104: 10k, Resistor_SMD:R_0402_1005Metric, F.Cu at (-82.9, 70.2)
- added R105: 31.6k, Resistor_SMD:R_0402_1005Metric, F.Cu at (-82.9, 72.2)
- added R106: 49, Resistor_SMD:R_0402_1005Metric, F.Cu at (-82.9, 74.1)
- added R107: 58.4k, Resistor_SMD:R_0402_1005Metric, F.Cu at (-82.9, 76.1)
- added R108: 10k, Resistor_SMD:R_0402_1005Metric, F.Cu at (-80.0, 64.2)
- added R109: 31.6k, Resistor_SMD:R_0402_1005Metric, F.Cu at (-80.0, 66.2)
- added R110: 49, Resistor_SMD:R_0402_1005Metric, F.Cu at (-80.0, 68.2)
- added R30: 464K, Resistor_SMD:R_0402_1005Metric, F.Cu at (209.3, 71.8)
- added R71: 33.2k, Resistor_SMD:R_0402_1005Metric, F.Cu at (209.3, 73.9)
- added R85: 47.5k, Resistor_SMD:R_0402_1005Metric, F.Cu at (209.3, 75.9)
- added R93: 453, Resistor_SMD:R_0402_1005Metric, F.Cu at (199.1, 74.3)
- added R94: 11.52, Resistor_SMD:R_0402_1005Metric, F.Cu at (199.1, 71.9)
- added R95: 58.4k, Resistor_SMD:R_0402_1005Metric, F.Cu at (-85.8, 66.2)
- added R96: 10k, Resistor_SMD:R_0402_1005Metric, F.Cu at (-85.8, 68.2)
- added R97: 31.6k, Resistor_SMD:R_0402_1005Metric, F.Cu at (-85.8, 70.2)
- added R98: 49, Resistor_SMD:R_0402_1005Metric, F.Cu at (-85.8, 72.2)
- added R99: 58.4k, Resistor_SMD:R_0402_1005Metric, F.Cu at (-85.8, 74.1)
- added U11: TPS259621DDAT, EFuse:SO-PP-DDA-8_TEX, F.Cu at (203.4, 73.1)
- JP8: footprint Jumper:SolderJumper-2_P1.3mm_Open_RoundedPad1.0x1.5mm -> iclr:SmallerSolderJP
- R45: value 90k -> 58.4k
- R48: value 31.7k -> 10k
- R51: value 10k -> 49
- R74: value 33.2K -> 31.6k
- R75: value 47.5K -> 58.4k
- R76: value 464K -> 10k
- R78: value 453 -> 31.6k
- R92: value 11.52 -> 49
- moved J1 326.0 mm to (228.1, 61.4)
- moved Y1 271.1 mm to (169.6, 87.6), turned to 90 degrees
- moved U9 270.7 mm to (202.6, 78.9)
- moved J12 268.2 mm to (199.4, 63.5), turned to 180 degrees
- moved J13 264.7 mm to (202.5, 96.6)
- moved R77 261.2 mm to (191.1, 75.4)
- moved D4 259.3 mm to (204.0, 82.6)
- moved J5 258.9 mm to (209.8, 60.9), turned to 90 degrees
- moved R91 257.0 mm to (162.2, 81.0)
- moved U1 255.6 mm to (167.6, 81.6), turned to 180 degrees
- moved C77 254.3 mm to (202.0, 86.5), turned to 90 degrees
- moved R79 253.5 mm to (207.2, 82.6), turned to 180 degrees
- moved Q2 249.1 mm to (191.1, 71.9)
- moved R89 246.9 mm to (194.1, 98.8), turned to -90 degrees
- moved J7 245.5 mm to (143.3, 69.4), turned to 90 degrees
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Connections:
- J7 pad 3: /pressure_sensor/AIN5N -> /pressure_sensor/AIN0N
- JP5 pad 3: Net-(JP5-B) -> /pressure_sensor/AIN0P
- JP8 pad 2: /pressure_sensor/AIN5N -> /pressure_sensor/AIN0N
- R45 pad 1: Net-(JP5-B) -> Net-(JP22-B)
- R45 pad 2: /pressure_sensor/AIN5P -> /pressure_sensor/AIN1P
- R48 pad 1: Net-(JP5-A) -> GND
- R48 pad 2: /pressure_sensor/AIN5P -> /pressure_sensor/AIN1P
- R51 pad 1: /pressure_sensor/AIN5P -> /pressure_sensor/AIN0P
- R51 pad 2: /pressure_sensor/AIN5N -> /pressure_sensor/AIN0N
- R74 pad 1: GND -> Net-(JP5-A)
- R74 pad 2: Net-(U8-EN/UVLO) -> Net-(JP20-C)
- R75 pad 1: GND -> Net-(JP20-B)
- R75 pad 2: GND -> /pressure_sensor/AIN0P
- R76 pad 1: Net-(U8-EN/UVLO) -> GND
- R76 pad 2: /Pyro/EFuse_In -> /pressure_sensor/AIN0P
- R78 pad 2: GND -> Net-(JP22-C)
- R92 pad 1: Net-(U8-*FLT) -> /pressure_sensor/AIN1P
- R92 pad 2: +3.3V -> /pressure_sensor/AIN1N
- U1 pad 24: /BuckP_EN -> /Pyro_IMON
Routing:
- net /pressure_sensor/AIN0N: track 0.00 -> 31.6 mm
- net /CAN-: track 10.3 -> 41.9 mm, vias 0 -> 1
- net /CAN+: track 10.3 -> 41.1 mm, vias 0 -> 1
- net /pressure_sensor/AIN1N: track 0.00 -> 26.4 mm
- net /pressure_sensor/AIN1P: track 0.00 -> 24.0 mm
- net /HSPI_SCLK: track 0.00 -> 18.8 mm
- net /HSPI_MISO: track 0.00 -> 18.8 mm
- net /HSPI_MOSI: track 0.00 -> 18.7 mm
- net /ADS_CS0: track 0.00 -> 18.7 mm
- net /Data+: track 9.66 -> 28.0 mm
- net /Data-: track 9.97 -> 28.0 mm
- net /ADS_CLK: track 0.00 -> 15.7 mm
- net /pressure_sensor/AIN0P: track 0.00 -> 10.4 mm
- net Net-(U11-OVLO/OVCSEL): track 0.00 -> 9.84 mm
- net Net-(J12-Pin_2): track 0.00 -> 9.81 mm
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- added copper zone on F.Cu, net /Pyro/PyroV
- added copper zone on F.Cu, net Net-(D3-K)
- added copper zone on F.Cu, net Net-(J12-Pin_2)
- added copper zone on F.Cu, net RBUS_uC_V
