File: can.kicad_sch (KiCad schematic)
At the start: 9 parts, among them U2 SN65HVD230

Commit message: Completed schematics
Parts:
- renumbered C15 to C14, C16 to C15, C17 to C16, R9 to R10, R10 to R11, R8 to R9
Changed lines of the file:
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@@
   (symbol (lib_id "power:GND") (at 134.62 99.06 0) (unit 1)
     (in_bom yes) (on_board yes) (dnp no) (fields_autoplaced)
-    (property "Reference" "#PWR026" (at 134.62 105.41 0)
+    (property "Reference" "#PWR025" (at 134.62 105.41 0)
       (effects (font (size 1.27 1.27)) hide)
     )
@@
       (project "EngineController"
         (path "/7db990e4-92e1-4f99-b4d2-435bbec1ba83/00000000-0000-0000-0000-000061942b9a"
-          (reference "#PWR026") (unit 1)
+          (reference "#PWR025") (unit 1)
         )
       )
@@
   (symbol (lib_id "power:+3.3V") (at 124.46 68.58 0) (unit 1)
     (in_bom yes) (on_board yes) (dnp no) (fields_autoplaced)
-    (property "Reference" "#PWR024" (at 124.46 72.39 0)
+    (property "Reference" "#PWR023" (at 124.46 72.39 0)
       (effects (font (size 1.27 1.27)) hide)
     )
@@
       (project "EngineController"
         (path "/7db990e4-92e1-4f99-b4d2-435bbec1ba83/00000000-0000-0000-0000-000061942b9a"
-          (reference "#PWR024") (unit 1)
+          (reference "#PWR023") (unit 1)
         )
       )
@@
   (symbol (lib_id "Device:C_Small") (at 127 71.12 0) (unit 1)
     (in_bom yes) (on_board yes) (dnp no) (fields_autoplaced)
-    (property "Reference" "C16" (at 129.54 69.8562 0)
+    (property "Reference" "C15" (at 129.54 69.8562 0)
       (effects (font (size 1.27 1.27)) (justify left))
     )
@@
       (project "EngineController"
         (path "/7db990e4-92e1-4f99-b4d2-435bbec1ba83/00000000-0000-0000-0000-000061942b9a"
-          (reference "C16") (unit 1)
+          (reference "C15") (unit 1)
         )
       )
@@
   (symbol (lib_id "power:GND") (at 177.8 88.9 0) (unit 1)
     (in_bom yes) (on_board yes) (dnp no) (fields_autoplaced)
-    (property "Reference" "#PWR027" (at 177.8 95.25 0)
+    (property "Reference" "#PWR026" (at 177.8 95.25 0)
       (effects (font (size 1.27 1.27)) hide)
     )
@@
       (project "EngineController"
         (path "/7db990e4-92e1-4f99-b4d2-435bbec1ba83/00000000-0000-0000-0000-000061942b9a"
-          (reference "#PWR027") (unit 1)
+          (reference "#PWR026") (unit 1)
         )
       )
@@
   (symbol (lib_id "Device:C_Small") (at 121.92 71.12 0) (unit 1)
     (in_bom yes) (on_board yes) (dnp no) (fields_autoplaced)
-    (property "Reference" "C15" (at 114.3 69.85 0)
+    (property "Reference" "C14" (at 114.3 69.85 0)
       (effects (font (size 1.27 1.27)) (justify left))
     )
@@
       (project "EngineController"
         (path "/7db990e4-92e1-4f99-b4d2-435bbec1ba83/00000000-0000-0000-0000-000061942b9a"
-          (reference "C15") (unit 1)
+          (reference "C14") (unit 1)
         )
       )
@@
   (symbol (lib_id "Device:R_Small") (at 124.46 95.25 0) (unit 1)
     (in_bom yes) (on_board yes) (dnp no)
-    (property "Reference" "R8" (at 118.11 93.98 0)
+    (property "Reference" "R9" (at 118.11 93.98 0)
       (effects (font (size 1.27 1.27)) (justify left))
     )
@@
       (project "EngineController"
         (path "/7db990e4-92e1-4f99-b4d2-435bbec1ba83/00000000-0000-0000-0000-000061942b9a"
-          (reference "R8") (unit 1)
+          (reference "R9") (unit 1)
         )
       )
@@
   (symbol (lib_id "Device:R") (at 167.64 93.98 0) (unit 1)
     (in_bom yes) (on_board yes) (dnp no) (fields_autoplaced)
-    (property "Reference" "R10" (at 162.56 92.71 0)
+    (property "Reference" "R11" (at 162.56 92.71 0)
       (effects (font (size 1.27 1.27)) (justify left))
     )
@@
       (project "EngineController"
         (path "/7db990e4-92e1-4f99-b4d2-435bbec1ba83/00000000-0000-0000-0000-000061942b9a"
+          (reference "R11") (unit 1)
+        )
+      )
+    )
+  )
+  (symbol (lib_id "Device:R") (at 167.64 83.82 0) (unit 1)
+    (in_bom yes) (on_board yes) (dnp no) (fields_autoplaced)
+    (property "Reference" "R10" (at 162.56 82.55 0)
+      (effects (font (size 1.27 1.27)) (justify left))
+    )
+    (property "Value" "60" (at 162.56 85.09 0)
+      (effects (font (size 1.27 1.27)) (justify left))
+    )
+    (property "Footprint" "Resistor_SMD:R_0603_1608Metric" (at 165.862 83.82 90)
+      (effects (font (size 1.27 1.27)) hide)
+    )
+    (property "Datasheet" "~" (at 167.64 83.82 0)
+      (effects (font (size 1.27 1.27)) hide)
+    )
+    (pin "1")
+    (pin "2")
+    (instances
+      (project "EngineController"
+        (path "/7db990e4-92e1-4f99-b4d2-435bbec1ba83/00000000-0000-0000-0000-000061942b9a"
           (reference "R10") (unit 1)
         )
@@
     )
   )
-  (symbol (lib_id "Device:R") (at 167.64 83.82 0) (unit 1)
-    (in_bom yes) (on_board yes) (dnp no) (fields_autoplaced)
-    (property "Reference" "R9" (at 162.56 82.55 0)
-      (effects (font (size 1.27 1.27)) (justify left))
-    )
-    (property "Value" "60" (at 162.56 85.09 0)
-      (effects (font (size 1.27 1.27)) (justify left))
-    )
-    (property "Footprint" "Resistor_SMD:R_0603_1608Metric" (at 165.862 83.82 90)
-      (effects (font (size 1.27 1.27)) hide)
-    )
-    (property "Datasheet" "~" (at 167.64 83.82 0)
-      (effects (font (size 1.27 1.27)) hide)
-    )
-    (pin "1")
-    (pin "2")
-    (instances
-      (project "EngineController"
-        (path "/7db990e4-92e1-4f99-b4d2-435bbec1ba83/00000000-0000-0000-0000-000061942b9a"
-          (reference "R9") (unit 1)
-        )
-      )
-    )
-  )
   (symbol (lib_id "Device:C") (at 171.45 88.9 90) (unit 1)
     (in_bom yes) (on_board yes) (dnp no) (fields_autoplaced)
-    (property "Reference" "C17" (at 171.45 82.55 90)
+    (property "Reference" "C16" (at 171.45 82.55 90)
       (effects (font (size 1.27 1.27)))
     )
@@
       (project "EngineController"
         (path "/7db990e4-92e1-4f99-b4d2-435bbec1ba83/00000000-0000-0000-0000-000061942b9a"
-          (reference "C17") (unit 1)
+          (reference "C16") (unit 1)
         )
       )
@@
   (symbol (lib_id "power:GND") (at 124.46 73.66 0) (unit 1)
     (in_bom yes) (on_board yes) (dnp no) (fields_autoplaced)
-    (property "Reference" "#PWR025" (at 124.46 80.01 0)
+    (property "Reference" "#PWR024" (at 124.46 80.01 0)
       (effects (font (size 1.27 1.27)) hide)
     )
@@
       (project "EngineController"
         (path "/7db990e4-92e1-4f99-b4d2-435bbec1ba83/00000000-0000-0000-0000-000061942b9a"
-          (reference "#PWR025") (unit 1)
-        )
-      )
+          (reference "#PWR024") (unit 1)
+        )
+      )

Commit message: More Based
Parts:
- renumbered R9 to R15, R10 to R16, R11 to R17
Changed lines of the file:
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@@
   (symbol (lib_id "power:GND") (at 134.62 99.06 0) (unit 1)
     (in_bom yes) (on_board yes) (dnp no) (fields_autoplaced)
-    (property "Reference" "#PWR025" (at 134.62 105.41 0)
+    (property "Reference" "#PWR035" (at 134.62 105.41 0)
       (effects (font (size 1.27 1.27)) hide)
     )
@@
       (project "Ricardo-Stark"
         (path "/7db990e4-92e1-4f99-b4d2-435bbec1ba83/00000000-0000-0000-0000-000061942b9a"
-          (reference "#PWR025") (unit 1)
+          (reference "#PWR035") (unit 1)
         )
       )
@@
   (symbol (lib_id "power:+3.3V") (at 124.46 68.58 0) (unit 1)
     (in_bom yes) (on_board yes) (dnp no) (fields_autoplaced)
-    (property "Reference" "#PWR023" (at 124.46 72.39 0)
+    (property "Reference" "#PWR033" (at 124.46 72.39 0)
       (effects (font (size 1.27 1.27)) hide)
     )
@@
       (project "Ricardo-Stark"
         (path "/7db990e4-92e1-4f99-b4d2-435bbec1ba83/00000000-0000-0000-0000-000061942b9a"
-          (reference "#PWR023") (unit 1)
+          (reference "#PWR033") (unit 1)
         )
       )
@@
   (symbol (lib_id "power:GND") (at 177.8 88.9 0) (unit 1)
     (in_bom yes) (on_board yes) (dnp no) (fields_autoplaced)
-    (property "Reference" "#PWR026" (at 177.8 95.25 0)
+    (property "Reference" "#PWR036" (at 177.8 95.25 0)
       (effects (font (size 1.27 1.27)) hide)
     )
@@
       (project "Ricardo-Stark"
         (path "/7db990e4-92e1-4f99-b4d2-435bbec1ba83/00000000-0000-0000-0000-000061942b9a"
-          (reference "#PWR026") (unit 1)
+          (reference "#PWR036") (unit 1)
         )
       )
@@
   (symbol (lib_id "Device:R_Small") (at 124.46 95.25 0) (unit 1)
     (in_bom yes) (on_board yes) (dnp no)
-    (property "Reference" "R9" (at 118.11 93.98 0)
+    (property "Reference" "R15" (at 118.11 93.98 0)
       (effects (font (size 1.27 1.27)) (justify left))
     )
@@
       (project "Ricardo-Stark"
         (path "/7db990e4-92e1-4f99-b4d2-435bbec1ba83/00000000-0000-0000-0000-000061942b9a"
-          (reference "R9") (unit 1)
+          (reference "R15") (unit 1)
         )
       )
@@
   (symbol (lib_id "Device:R") (at 167.64 93.98 0) (unit 1)
     (in_bom yes) (on_board yes) (dnp no) (fields_autoplaced)
-    (property "Reference" "R11" (at 162.56 92.71 0)
+    (property "Reference" "R17" (at 162.56 92.71 0)
       (effects (font (size 1.27 1.27)) (justify left))
     )
@@
       (project "Ricardo-Stark"
         (path "/7db990e4-92e1-4f99-b4d2-435bbec1ba83/00000000-0000-0000-0000-000061942b9a"
-          (reference "R11") (unit 1)
+          (reference "R17") (unit 1)
         )
       )
@@
   (symbol (lib_id "Device:R") (at 167.64 83.82 0) (unit 1)
     (in_bom yes) (on_board yes) (dnp no) (fields_autoplaced)
-    (property "Reference" "R10" (at 162.56 82.55 0)
+    (property "Reference" "R16" (at 162.56 82.55 0)
       (effects (font (size 1.27 1.27)) (justify left))
     )
@@
       (project "Ricardo-Stark"
         (path "/7db990e4-92e1-4f99-b4d2-435bbec1ba83/00000000-0000-0000-0000-000061942b9a"
-          (reference "R10") (unit 1)
+          (reference "R16") (unit 1)
         )
       )
@@
   (symbol (lib_id "power:GND") (at 124.46 73.66 0) (unit 1)
     (in_bom yes) (on_board yes) (dnp no) (fields_autoplaced)
-    (property "Reference" "#PWR024" (at 124.46 80.01 0)
+    (property "Reference" "#PWR034" (at 124.46 80.01 0)
       (effects (font (size 1.27 1.27)) hide)
     )
@@
       (project "Ricardo-Stark"
         (path "/7db990e4-92e1-4f99-b4d2-435bbec1ba83/00000000-0000-0000-0000-000061942b9a"
-          (reference "#PWR024") (unit 1)
-        )
-      )
+          (reference "#PWR034") (unit 1)
+        )
+      )

Commit message: Take 3
Parts:
- JP1: footprint Jumper:SolderJumper-2_P1.3mm_Open_RoundedPad1.0x1.5mm -> iclr:SmallerSolderJP
Changed lines of the file:
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@@
       (effects (font (size 1.27 1.27)))
     )
-    (property "Footprint" "Jumper:SolderJumper-2_P1.3mm_Open_RoundedPad1.0x1.5mm" (at 157.48 88.9 0)
+    (property "Footprint" "iclr:SmallerSolderJP" (at 157.48 88.9 0)
       (effects (font (size 1.27 1.27)) hide)
     )
