File: usb.kicad_sch (KiCad schematic)
At the start: 8 parts, among them J2 USB_C_Receptacle_USB2.0

Commit message: Completed schematics
Parts:
- renumbered R11 to R12, R12 to R13, R13 to R14, TP1 to TP3, TP2 to TP4
Changed lines of the file:
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@@
   (junction (at 115.57 102.87) (diameter 0) (color 0 0 0 0)
+  )
+  (junction (at 152.4 92.71) (diameter 0) (color 0 0 0 0)
   )
   (no_connect (at 115.57 119.38))
@@
   (symbol (lib_id "power:GND") (at 127 96.52 90) (unit 1)
     (in_bom yes) (on_board yes) (dnp no)
-    (property "Reference" "#PWR031" (at 133.35 96.52 0)
+    (property "Reference" "#PWR029" (at 133.35 96.52 0)
       (effects (font (size 1.27 1.27)) hide)
     )
@@
       (project "EngineController"
         (path "/7db990e4-92e1-4f99-b4d2-435bbec1ba83/00000000-0000-0000-0000-000061925999"
-          (reference "#PWR031") (unit 1)
+          (reference "#PWR029") (unit 1)
         )
       )
@@
   (symbol (lib_id "Device:R_Small") (at 123.19 99.06 270) (unit 1)
     (in_bom yes) (on_board yes) (dnp no)
-    (property "Reference" "R12" (at 129.54 100.33 90)
+    (property "Reference" "R13" (at 129.54 100.33 90)
       (effects (font (size 1.27 1.27)))
     )
@@
       (project "EngineController"
         (path "/7db990e4-92e1-4f99-b4d2-435bbec1ba83/00000000-0000-0000-0000-000061925999"
+          (reference "R13") (unit 1)
+        )
+      )
+    )
+  )
+  (symbol (lib_id "Device:R_Small") (at 123.19 93.98 90) (unit 1)
+    (in_bom yes) (on_board yes) (dnp no)
+    (property "Reference" "R12" (at 123.19 89.0016 90)
+      (effects (font (size 1.27 1.27)))
+    )
+    (property "Value" "5.1k" (at 123.19 91.313 90)
+      (effects (font (size 1.27 1.27)))
+    )
+    (property "Footprint" "Resistor_SMD:R_0402_1005Metric" (at 123.19 93.98 0)
+      (effects (font (size 1.27 1.27)) hide)
+    )
+    (property "Datasheet" "~" (at 123.19 93.98 0)
+      (effects (font (size 1.27 1.27)) hide)
+    )
+    (pin "1")
+    (pin "2")
+    (instances
+      (project "EngineController"
+        (path "/7db990e4-92e1-4f99-b4d2-435bbec1ba83/00000000-0000-0000-0000-000061925999"
           (reference "R12") (unit 1)
         )
@@
     )
   )
-  (symbol (lib_id "Device:R_Small") (at 123.19 93.98 90) (unit 1)
-    (in_bom yes) (on_board yes) (dnp no)
-    (property "Reference" "R11" (at 123.19 89.0016 90)
-      (effects (font (size 1.27 1.27)))
-    )
-    (property "Value" "5.1k" (at 123.19 91.313 90)
-      (effects (font (size 1.27 1.27)))
-    )
-    (property "Footprint" "Resistor_SMD:R_0402_1005Metric" (at 123.19 93.98 0)
-      (effects (font (size 1.27 1.27)) hide)
-    )
-    (property "Datasheet" "~" (at 123.19 93.98 0)
-      (effects (font (size 1.27 1.27)) hide)
-    )
-    (pin "1")
-    (pin "2")
-    (instances
-      (project "EngineController"
-        (path "/7db990e4-92e1-4f99-b4d2-435bbec1ba83/00000000-0000-0000-0000-000061925999"
-          (reference "R11") (unit 1)
-        )
-      )
-    )
-  )
   (symbol (lib_id "power:GND") (at 96.52 130.81 0) (unit 1)
     (in_bom yes) (on_board yes) (dnp no)
-    (property "Reference" "#PWR029" (at 96.52 137.16 0)
+    (property "Reference" "#PWR027" (at 96.52 137.16 0)
       (effects (font (size 1.27 1.27)) hide)
     )
@@
       (project "EngineController"
         (path "/7db990e4-92e1-4f99-b4d2-435bbec1ba83/00000000-0000-0000-0000-000061925999"
-          (reference "#PWR029") (unit 1)
+          (reference "#PWR027") (unit 1)
         )
       )
@@
   (symbol (lib_id "power:GND") (at 132.08 144.78 0) (unit 1)
     (in_bom yes) (on_board yes) (dnp no)
-    (property "Reference" "#PWR032" (at 132.08 151.13 0)
+    (property "Reference" "#PWR030" (at 132.08 151.13 0)
       (effects (font (size 1.27 1.27)) hide)
     )
@@
       (project "EngineController"
         (path "/7db990e4-92e1-4f99-b4d2-435bbec1ba83/00000000-0000-0000-0000-000061925999"
-          (reference "#PWR032") (unit 1)
+          (reference "#PWR030") (unit 1)
         )
       )
@@
   (symbol (lib_id "power:VBUS") (at 116.84 85.09 0) (unit 1)
     (in_bom yes) (on_board yes) (dnp no)
-    (property "Reference" "#PWR030" (at 116.84 88.9 0)
+    (property "Reference" "#PWR028" (at 116.84 88.9 0)
       (effects (font (size 1.27 1.27)) hide)
     )
@@
       (project "EngineController"
         (path "/7db990e4-92e1-4f99-b4d2-435bbec1ba83/00000000-0000-0000-0000-000061925999"
-          (reference "#PWR030") (unit 1)
+          (reference "#PWR028") (unit 1)
         )
       )
@@
   (symbol (lib_id "Connector:TestPoint") (at 52.07 99.06 270) (unit 1)
     (in_bom yes) (on_board yes) (dnp no)
-    (property "Reference" "TP1" (at 56.8452 97.8916 90)
+    (property "Reference" "TP3" (at 56.8452 97.8916 90)
       (effects (font (size 1.27 1.27)) (justify left))
     )
@@
       (project "EngineController"
         (path "/7db990e4-92e1-4f99-b4d2-435bbec1ba83/00000000-0000-0000-0000-000061925999"
-          (reference "TP1") (unit 1)
+          (reference "TP3") (unit 1)
         )
       )
@@
   (symbol (lib_id "Connector:TestPoint") (at 52.07 104.14 270) (unit 1)
     (in_bom yes) (on_board yes) (dnp no)
-    (property "Reference" "TP2" (at 56.8452 102.9716 90)
+    (property "Reference" "TP4" (at 56.8452 102.9716 90)
       (effects (font (size 1.27 1.27)) (justify left))
     )
@@
       (project "EngineController"
         (path "/7db990e4-92e1-4f99-b4d2-435bbec1ba83/00000000-0000-0000-0000-000061925999"
-          (reference "TP2") (unit 1)
+          (reference "TP4") (unit 1)
         )
       )
@@
   (symbol (lib_id "Device:R_Small") (at 154.94 92.71 90) (unit 1)
     (in_bom yes) (on_board yes) (dnp no)
-    (property "Reference" "R13" (at 154.94 95.3516 90)
+    (property "Reference" "R14" (at 154.94 95.3516 90)
       (effects (font (size 1.27 1.27)))
     )
@@
       (project "EngineController"
         (path "/7db990e4-92e1-4f99-b4d2-435bbec1ba83/00000000-0000-0000-0000-000061925999"
-          (reference "R13") (unit 1)
+          (reference "R14") (unit 1)
         )
       )
@@
   (symbol (lib_id "power:GND") (at 165.1 92.71 90) (unit 1)
     (in_bom yes) (on_board yes) (dnp no)
-    (property "Reference" "#PWR034" (at 171.45 92.71 0)
+    (property "Reference" "#PWR032" (at 171.45 92.71 0)
       (effects (font (size 1.27 1.27)) hide)
     )
@@
       (project "EngineController"
         (path "/7db990e4-92e1-4f99-b4d2-435bbec1ba83/00000000-0000-0000-0000-000061925999"
-          (reference "#PWR034") (unit 1)
+          (reference "#PWR032") (unit 1)
         )
       )
@@
   (symbol (lib_id "power:VBUS") (at 152.4 92.71 90) (unit 1)
     (in_bom yes) (on_board yes) (dnp no)
-    (property "Reference" "#PWR033" (at 156.21 92.71 0)
+    (property "Reference" "#PWR031" (at 156.21 92.71 0)
       (effects (font (size 1.27 1.27)) hide)
     )
@@
       (project "EngineController"
         (path "/7db990e4-92e1-4f99-b4d2-435bbec1ba83/00000000-0000-0000-0000-000061925999"
-          (reference "#PWR033") (unit 1)
-        )
-      )
+          (reference "#PWR031") (unit 1)
+        )
+      )
+    )
+  )
+  (symbol (lib_id "power:PWR_FLAG") (at 152.4 92.71 0) (unit 1)
+    (in_bom yes) (on_board yes) (dnp no) (fields_autoplaced)
+    (property "Reference" "#FLG013" (at 152.4 90.805 0)
+      (effects (font (size 1.27 1.27)) hide)
+    )
+    (property "Value" "PWR_FLAG" (at 152.4 87.63 0)
+      (effects (font (size 1.27 1.27)))
+    )
+    (property "Footprint" "" (at 152.4 92.71 0)
+      (effects (font (size 1.27 1.27)) hide)
+    )
+    (property "Datasheet" "~" (at 152.4 92.71 0)
+      (effects (font (size 1.27 1.27)) hide)
+    )
+    (pin "1")
+    (instances
+      (project "EngineController"
+        (path "/7db990e4-92e1-4f99-b4d2-435bbec1ba83/00000000-0000-0000-0000-000061925999"
+          (reference "#FLG013") (unit 1)
+        )
+      )

Commit message: More Based
Parts:
- renumbered R12 to R18, R13 to R19, R14 to R20
Changed lines of the file:
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@@
   (symbol (lib_id "power:GND") (at 127 96.52 90) (unit 1)
     (in_bom yes) (on_board yes) (dnp no)
-    (property "Reference" "#PWR029" (at 133.35 96.52 0)
+    (property "Reference" "#PWR039" (at 133.35 96.52 0)
       (effects (font (size 1.27 1.27)) hide)
     )
@@
       (project "Ricardo-Stark"
         (path "/7db990e4-92e1-4f99-b4d2-435bbec1ba83/00000000-0000-0000-0000-000061925999"
-          (reference "#PWR029") (unit 1)
+          (reference "#PWR039") (unit 1)
         )
       )
@@
   (symbol (lib_id "Device:R_Small") (at 123.19 99.06 270) (unit 1)
     (in_bom yes) (on_board yes) (dnp no)
-    (property "Reference" "R13" (at 129.54 100.33 90)
+    (property "Reference" "R19" (at 129.54 100.33 90)
       (effects (font (size 1.27 1.27)))
     )
@@
       (project "Ricardo-Stark"
         (path "/7db990e4-92e1-4f99-b4d2-435bbec1ba83/00000000-0000-0000-0000-000061925999"
-          (reference "R13") (unit 1)
+          (reference "R19") (unit 1)
         )
       )
@@
   (symbol (lib_id "Device:R_Small") (at 123.19 93.98 90) (unit 1)
     (in_bom yes) (on_board yes) (dnp no)
-    (property "Reference" "R12" (at 123.19 89.0016 90)
+    (property "Reference" "R18" (at 123.19 89.0016 90)
       (effects (font (size 1.27 1.27)))
     )
@@
       (project "Ricardo-Stark"
         (path "/7db990e4-92e1-4f99-b4d2-435bbec1ba83/00000000-0000-0000-0000-000061925999"
-          (reference "R12") (unit 1)
+          (reference "R18") (unit 1)
         )
       )
@@
   (symbol (lib_id "power:GND") (at 96.52 130.81 0) (unit 1)
     (in_bom yes) (on_board yes) (dnp no)
-    (property "Reference" "#PWR027" (at 96.52 137.16 0)
+    (property "Reference" "#PWR037" (at 96.52 137.16 0)
       (effects (font (size 1.27 1.27)) hide)
     )
@@
       (project "Ricardo-Stark"
         (path "/7db990e4-92e1-4f99-b4d2-435bbec1ba83/00000000-0000-0000-0000-000061925999"
-          (reference "#PWR027") (unit 1)
+          (reference "#PWR037") (unit 1)
         )
       )
@@
   (symbol (lib_id "power:GND") (at 132.08 144.78 0) (unit 1)
     (in_bom yes) (on_board yes) (dnp no)
-    (property "Reference" "#PWR030" (at 132.08 151.13 0)
+    (property "Reference" "#PWR040" (at 132.08 151.13 0)
       (effects (font (size 1.27 1.27)) hide)
     )
@@
       (project "Ricardo-Stark"
         (path "/7db990e4-92e1-4f99-b4d2-435bbec1ba83/00000000-0000-0000-0000-000061925999"
-          (reference "#PWR030") (unit 1)
+          (reference "#PWR040") (unit 1)
         )
       )
@@
   (symbol (lib_id "power:VBUS") (at 116.84 85.09 0) (unit 1)
     (in_bom yes) (on_board yes) (dnp no)
-    (property "Reference" "#PWR028" (at 116.84 88.9 0)
+    (property "Reference" "#PWR038" (at 116.84 88.9 0)
       (effects (font (size 1.27 1.27)) hide)
     )
@@
       (project "Ricardo-Stark"
         (path "/7db990e4-92e1-4f99-b4d2-435bbec1ba83/00000000-0000-0000-0000-000061925999"
-          (reference "#PWR028") (unit 1)
+          (reference "#PWR038") (unit 1)
         )
       )
@@
   (symbol (lib_id "Device:R_Small") (at 154.94 92.71 90) (unit 1)
     (in_bom yes) (on_board yes) (dnp no)
-    (property "Reference" "R14" (at 154.94 95.3516 90)
+    (property "Reference" "R20" (at 154.94 95.3516 90)
       (effects (font (size 1.27 1.27)))
     )
@@
       (project "Ricardo-Stark"
         (path "/7db990e4-92e1-4f99-b4d2-435bbec1ba83/00000000-0000-0000-0000-000061925999"
-          (reference "R14") (unit 1)
+          (reference "R20") (unit 1)
         )
       )
@@
   (symbol (lib_id "power:GND") (at 165.1 92.71 90) (unit 1)
     (in_bom yes) (on_board yes) (dnp no)
-    (property "Reference" "#PWR032" (at 171.45 92.71 0)
+    (property "Reference" "#PWR042" (at 171.45 92.71 0)
       (effects (font (size 1.27 1.27)) hide)
     )
@@
       (project "Ricardo-Stark"
         (path "/7db990e4-92e1-4f99-b4d2-435bbec1ba83/00000000-0000-0000-0000-000061925999"
-          (reference "#PWR032") (unit 1)
+          (reference "#PWR042") (unit 1)
         )
       )
@@
   (symbol (lib_id "power:VBUS") (at 152.4 92.71 90) (unit 1)
     (in_bom yes) (on_board yes) (dnp no)
-    (property "Reference" "#PWR031" (at 156.21 92.71 0)
+    (property "Reference" "#PWR041" (at 156.21 92.71 0)
       (effects (font (size 1.27 1.27)) hide)
     )
@@
       (project "Ricardo-Stark"
         (path "/7db990e4-92e1-4f99-b4d2-435bbec1ba83/00000000-0000-0000-0000-000061925999"
-          (reference "#PWR031") (unit 1)
+          (reference "#PWR041") (unit 1)
         )
       )
@@
   (symbol (lib_id "power:PWR_FLAG") (at 152.4 92.71 0) (unit 1)
     (in_bom yes) (on_board yes) (dnp no) (fields_autoplaced)
-    (property "Reference" "#FLG013" (at 152.4 90.805 0)
+    (property "Reference" "#FLG03" (at 152.4 90.805 0)
       (effects (font (size 1.27 1.27)) hide)
     )
@@
       (project "Ricardo-Stark"
         (path "/7db990e4-92e1-4f99-b4d2-435bbec1ba83/00000000-0000-0000-0000-000061925999"
-          (reference "#FLG013") (unit 1)
-        )
-      )
+          (reference "#FLG03") (unit 1)
+        )
+      )
