File: actuators.kicad_sch (KiCad schematic)
At the start: 5 parts, among them J3 ServoCH1, J4 ServoCH2

Commit message: Finished schematic
Parts:
- added J2: GPIO Breakout, Connector_PinSocket_2.54mm:PinSocket_2x04_P2.54mm_Vertical, symbol Connector:Conn_01x08_Female
- added R28, R29, R30, R31, R32, R33: DNP, Resistor_SMD:R_0402_1005Metric, symbol Device:R_Small
Connections:
- net GND: now also J2.1 (Pin_1)
- new net +3V3: J2.5 (Pin_5), R28.1, R29.1, R30.1, R31.1, R32.1, R33.1
- new net GPIO0: J2.2 (Pin_2), R31.2
- new net GPIO1: J2.3 (Pin_3), R29.2
- new net GPIO2: J2.4 (Pin_4), R28.2
- new net GPIO3: J2.6 (Pin_6), R30.2
- new net GPIO4: J2.7 (Pin_7), R32.2
- new net GPIO5: J2.8 (Pin_8), R33.2

Commit message: Commit
Connections:
- net GPIO0 renamed GPIO9
- net GPIO1 renamed GPIO8
- net GPIO2 renamed GPIO7
- net GPIO3 renamed GPIO6
Changed lines of the file:
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@@
-    (effects (font (size 1.27 1.27)) (justify right bottom))
-  )
-  (label "GPIO0" (at 191.008 102.87 270) (fields_autoplaced)
-    (effects (font (size 1.27 1.27)) (justify right bottom))
-  )
-  (label "GPIO1" (at 227.838 71.12 180) (fields_autoplaced)
-    (effects (font (size 1.27 1.27)) (justify right bottom))
-  )
-  (label "GPIO2" (at 227.838 73.66 180) (fields_autoplaced)
     (effects (font (size 1.27 1.27)) (justify right bottom))
   )
@@
     (effects (font (size 1.27 1.27)) (justify right bottom))
   )
-  (label "GPIO0" (at 227.838 68.58 180) (fields_autoplaced)
-    (effects (font (size 1.27 1.27)) (justify right bottom))
+  (hierarchical_label "GPIO9" (shape input) (at 191.008 102.87 270) (fields_autoplaced)
+    (effects (font (size 1.27 1.27)) (justify right))
   )
-  (label "GPIO4" (at 227.838 81.28 180) (fields_autoplaced)
-    (effects (font (size 1.27 1.27)) (justify right bottom))
+  (hierarchical_label "GPIO7" (shape input) (at 227.838 73.66 180) (fields_autoplaced)
+    (effects (font (size 1.27 1.27)) (justify right))
   )
-  (label "GPIO3" (at 212.598 102.87 270) (fields_autoplaced)
-    (effects (font (size 1.27 1.27)) (justify right bottom))
-  )
-  (label "GPIO4" (at 218.948 102.87 270) (fields_autoplaced)
-    (effects (font (size 1.27 1.27)) (justify right bottom))
-  )
-  (label "GPIO2" (at 204.978 102.87 270) (fields_autoplaced)
-    (effects (font (size 1.27 1.27)) (justify right bottom))
-  )
-  (label "GPIO5" (at 226.568 102.87 270) (fields_autoplaced)
-    (effects (font (size 1.27 1.27)) (justify right bottom))
-  )
-  (label "GPIO3" (at 227.838 78.74 180) (fields_autoplaced)
-    (effects (font (size 1.27 1.27)) (justify right bottom))
-  )
-  (label "GPIO5" (at 227.838 83.82 180) (fields_autoplaced)
-    (effects (font (size 1.27 1.27)) (justify right bottom))
-  )
-  (label "GPIO1" (at 197.358 102.87 270) (fields_autoplaced)
-    (effects (font (size 1.27 1.27)) (justify right bottom))
+  (hierarchical_label "GPIO4" (shape input) (at 218.948 102.87 270) (fields_autoplaced)
+    (effects (font (size 1.27 1.27)) (justify right))
   )
   (hierarchical_label "SERVO1" (shape bidirectional) (at 153.67 68.58 180) (fields_autoplaced)
+    (effects (font (size 1.27 1.27)) (justify right))
+  )
+  (hierarchical_label "GPIO6" (shape input) (at 227.838 78.74 180) (fields_autoplaced)
+    (effects (font (size 1.27 1.27)) (justify right))
+  )
+  (hierarchical_label "GPIO8" (shape input) (at 227.838 71.12 180) (fields_autoplaced)
+    (effects (font (size 1.27 1.27)) (justify right))
+  )
+  (hierarchical_label "GPIO4" (shape input) (at 227.838 81.28 180) (fields_autoplaced)
+    (effects (font (size 1.27 1.27)) (justify right))
+  )
+  (hierarchical_label "GPIO7" (shape input) (at 204.978 102.87 270) (fields_autoplaced)
+    (effects (font (size 1.27 1.27)) (justify right))
+  )
+  (hierarchical_label "GPIO8" (shape input) (at 197.358 102.87 270) (fields_autoplaced)
+    (effects (font (size 1.27 1.27)) (justify right))
+  )
+  (hierarchical_label "GPIO5" (shape input) (at 227.838 83.82 180) (fields_autoplaced)
     (effects (font (size 1.27 1.27)) (justify right))
   )
@@
     (effects (font (size 1.27 1.27)) (justify right))
   )
+  (hierarchical_label "GPIO9" (shape input) (at 227.838 68.58 180) (fields_autoplaced)
+    (effects (font (size 1.27 1.27)) (justify right))
+  )
+  (hierarchical_label "GPIO5" (shape input) (at 226.568 102.87 270) (fields_autoplaced)
+    (effects (font (size 1.27 1.27)) (justify right))
+  )
   (hierarchical_label "SERVO2" (shape bidirectional) (at 153.67 83.82 180) (fields_autoplaced)
     (effects (font (size 1.27 1.27)) (justify right))
   )
+  (hierarchical_label "GPIO6" (shape input) (at 212.598 102.87 270) (fields_autoplaced)
+    (effects (font (size 1.27 1.27)) (justify right))
+  )

Commit message: review changes
Parts:
- renumbered C12 to C36, J2 to J5, R26 to R34, R27 to R35, R31 to R36, R29 to R37, R28 to R38, R30 to R39, R32 to R40, R33 to R41

Commit message: 5v breakout
Parts:
- J5: footprint Connector_PinSocket_2.54mm:PinSocket_2x04_P2.54mm_Vertical -> Connector_PinSocket_2.54mm:PinSocket_2x05_P2.54mm_Vertical; symbol Connector:Conn_01x08_Female -> Connector:Conn_01x10_Socket
Connections:
- new net 5V: J5.9 (Pin_9)
- no-connect marks 0 -> 1
Changed lines of the file:
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@@
 		(color 0 0 0 0)
+	)
+	(no_connect
+		(at 227.838 86.36)
 	)
 	(wire
@@
 	(hierarchical_label "GPIO7"
 		(shape input)
-		(at 227.838 73.66 180)
+		(at 227.838 71.12 180)
 		(fields_autoplaced yes)
 		(effects
@@
 	(hierarchical_label "GPIO6"
 		(shape input)
-		(at 227.838 78.74 180)
+		(at 227.838 76.2 180)
 		(fields_autoplaced yes)
 		(effects
@@
 	(hierarchical_label "GPIO8"
 		(shape input)
-		(at 227.838 71.12 180)
+		(at 227.838 68.58 180)
+		(fields_autoplaced yes)
+		(effects
+			(font
+				(size 1.27 1.27)
+			)
+			(justify right)
+		)
+	)
+	(hierarchical_label "5V"
+		(shape output)
+		(at 227.838 83.82 180)
 		(fields_autoplaced yes)
 		(effects
@@
 	(hierarchical_label "GPIO4"
 		(shape input)
-		(at 227.838 81.28 180)
+		(at 227.838 78.74 180)
 		(fields_autoplaced yes)
 		(effects
@@
 	(hierarchical_label "GPIO5"
 		(shape input)
-		(at 227.838 83.82 180)
+		(at 227.838 81.28 180)
 		(fields_autoplaced yes)
 		(effects
@@
 	(hierarchical_label "GPIO9"
 		(shape input)
-		(at 227.838 68.58 180)
+		(at 227.838 66.04 180)
 		(fields_autoplaced yes)
 		(effects
@@
 	)
 	(symbol
-		(lib_id "Connector:Conn_01x08_Female")
+		(lib_id "Connector:Conn_01x10_Socket")
 		(at 232.918 73.66 0)
 		(unit 1)
@@
 			)
 		)
-		(property "Footprint" "Connector_PinSocket_2.54mm:PinSocket_2x04_P2.54mm_Vertical"
+		(property "Footprint" "Connector_PinSocket_2.54mm:PinSocket_2x05_P2.54mm_Vertical"
 			(at 232.918 73.66 0)
 			(effects
@@
 			)
 		)
-		(property "Description" ""
+		(property "Description" "Generic connector, single row, 01x10, script generated"
 			(at 232.918 73.66 0)
 			(effects
@@
 		)
 		(pin "8"
+		)
+		(pin "9"
+		)
+		(pin "10"
 		)
 		(instances
@@
 	(symbol
 		(lib_id "power:GND")
+		(at 227.838 63.5 270)
+		(unit 1)
+		(exclude_from_sim no)
+		(in_bom yes)
+		(on_board yes)
+		(dnp no)
+		(fields_autoplaced yes)
+		(property "Reference" "#PWR093"
+			(at 221.488 63.5 0)
+			(effects
+				(font
+					(size 1.27 1.27)
+				)
+				(hide yes)
+			)
+		)
+		(property "Value" "GND"
+			(at 224.6631 63.9338 90)
+			(effects
+				(font
+					(size 1.27 1.27)
+				)
+				(justify right)
+			)
+		)
+		(property "Footprint" ""
+			(at 227.838 63.5 0)
+			(effects
+				(font
+					(size 1.27 1.27)
+				)
+				(hide yes)
+			)
+		)
+		(property "Datasheet" ""
+			(at 227.838 63.5 0)
+			(effects
+				(font
+					(size 1.27 1.27)
+				)
+				(hide yes)
+			)
+		)
+		(property "Description" ""
+			(at 227.838 63.5 0)
+			(effects
+				(font
+					(size 1.27 1.27)
+				)
+				(hide yes)
+			)
+		)
+		(pin "1"
+		)
+		(instances
+			(project "Ricardo-Stark"
+				(path "/7db990e4-92e1-4f99-b4d2-435bbec1ba83/5f0880ee-ff3b-4d6c-b43c-55333f7e65e0"
+					(reference "#PWR093")
+					(unit 1)
+				)
+			)
+		)
+	)
+	(symbol
+		(lib_id "power:GND")
 		(at 157.48 113.03 0)
 		(unit 1)
@@
 	(symbol
 		(lib_id "power:+3.3V")
-		(at 227.838 76.2 90)
-		(unit 1)
-		(exclude_from_sim no)
-		(in_bom yes)
-		(on_board yes)
-		(dnp no)
-		(fields_autoplaced yes)
+		(at 227.838 73.66 90)
+		(unit 1)
+		(exclude_from_sim no)
+		(in_bom yes)
+		(on_board yes)
+		(dnp no)
 		(property "Reference" "#PWR086"
-			(at 231.648 76.2 0)
+			(at 231.648 73.66 0)
 			(effects
 				(font
@@
 		)
 		(property "Value" "+3V3"
-			(at 224.663 76.6338 90)
+			(at 224.663 74.0938 90)
 			(effects
 				(font
@@
 		)
 		(property "Footprint" ""
-			(at 227.838 76.2 0)
+			(at 227.838 73.66 0)
 			(effects
 				(font
@@
 		)
 		(property "Datasheet" ""
-			(at 227.838 76.2 0)
-			(effects
-				(font
-					(size 1.27 1.27)
-				)
-				(hide yes)
-			)
-		)
-		(property "Description" ""
-			(at 227.838 76.2 0)
+			(at 227.838 73.66 0)
+			(effects
+				(font
+					(size 1.27 1.27)
+				)
+				(hide yes)
+			)
+		)
+		(property "Description" ""
+			(at 227.838 73.66 0)
 			(effects
 				(font
@@
 					(unit 1)
 				)
-			)
-		)
-	)
-	(symbol
-		(lib_id "power:GND")
-		(at 227.838 66.04 270)
-		(unit 1)
-		(exclude_from_sim no)
-		(in_bom yes)
-		(on_board yes)
-		(dnp no)
-		(fields_autoplaced yes)
-		(property "Reference" "#PWR085"
-			(at 221.488 66.04 0)
-			(effects
-				(font
-					(size 1.27 1.27)
-				)
-				(hide yes)
-			)
-		)
-		(property "Value" "GND"
-			(at 224.6631 66.4738 90)
-			(effects
-				(font
-					(size 1.27 1.27)
-				)
-				(justify right)
-			)
-		)
-		(property "Footprint" ""
-			(at 227.838 66.04 0)
-			(effects
-				(font
-					(size 1.27 1.27)
-				)
-				(hide yes)
-			)
-		)
-		(property "Datasheet" ""
-			(at 227.838 66.04 0)
-			(effects
-				(font
-					(size 1.27 1.27)
-				)
-				(hide yes)
-			)
-		)
-		(property "Description" ""
-			(at 227.838 66.04 0)
-			(effects
-				(font
-					(size 1.27 1.27)
-				)
-				(hide yes)
-			)
-		)
-		(pin "1"
-		)
-		(instances
-			(project "Ricardo-Stark"
-				(path "/7db990e4-92e1-4f99-b4d2-435bbec1ba83/5f0880ee-ff3b-4d6c-b43c-55333f7e65e0"
-					(reference "#PWR085")
-					(unit 1)
-				)
