File: buckCkicad_sch.kicad_sch (KiCad schematic)
At the start: 25 parts, among them Q1 SSM3K15AMFV,L3F, U6 SiC437BED-T1-GE3

Commit message: Most Review 1 changes made
Parts:
- C29: value 47uF -> 68uF
- C31, C33: value 47uF -> 220uF
Changed lines of the file:
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@@
       (effects (font (size 1.27 1.27)) (justify left))
     )
-    (property "Value" "47uF" (at 85.09 119.3863 0)
+    (property "Value" "68uF" (at 85.09 119.3863 0)
       (effects (font (size 1.27 1.27)) (justify left))
     )
@@
       (effects (font (size 1.27 1.27)) (justify left))
     )
-    (property "Value" "47uF" (at 102.87 119.3863 0)
+    (property "Value" "220uF" (at 102.87 119.3863 0)
       (effects (font (size 1.27 1.27)) (justify left))
     )
@@
       (effects (font (size 1.27 1.27)) (justify left))
     )
-    (property "Value" "47uF" (at 93.98 119.3863 0)
-      (effects (font (size 1.27 1.27)) (justify left))
-    )
+    (property "Value" "220uF" (at 93.98 119.3863 0)
+      (effects (font (size 1.27 1.27)) (justify left))
+    )

Commit message: Review 1 Changes Complete
Connections:
- net +12V renamed DeployV
Changed lines of the file:
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@@
     (effects (font (size 1.27 1.27)) (justify right bottom))
+  )
+  (global_label "DeployV" (shape bidirectional) (at 66.04 27.94 90) (fields_autoplaced)
+    (effects (font (size 1.27 1.27)) (justify left))
+    (property "Intersheetrefs" "${INTERSHEET_REFS}" (at 66.04 17.2785 90)
+      (effects (font (size 1.27 1.27)) (justify left) hide)
+    )
   )
   (hierarchical_label "BUCKC_EN" (shape input) (at 132.08 119.38 180) (fields_autoplaced)
@@
         )
       )
-    )
-  )
-  (symbol (lib_id "power:+12V") (at 66.04 27.94 0) (unit 1)
-    (in_bom yes) (on_board yes) (dnp no) (fields_autoplaced)
-    (property "Reference" "#PWR063" (at 66.04 31.75 0)
-      (effects (font (size 1.27 1.27)) hide)
-    )
-    (property "Value" "+12V" (at 66.04 24.3642 0)
-      (effects (font (size 1.27 1.27)))
-    )
-    (property "Footprint" "" (at 66.04 27.94 0)
-      (effects (font (size 1.27 1.27)) hide)
-    )
-    (property "Datasheet" "" (at 66.04 27.94 0)
-      (effects (font (size 1.27 1.27)) hide)
-    )
-    (pin "1")
-    (instances
-      (project "Ricardo-Stark"
-        (path "/7db990e4-92e1-4f99-b4d2-435bbec1ba83/6c17bf58-bab3-4fa6-ad33-cca9e388d73c"
-          (reference "#PWR063") (unit 1)
-        )
-      )

Commit message: Take 3
Parts:
- removed Q1: SSM3K15AMFV,L3F, Package_TO_SOT_SMD:SOT-723, symbol Device:Q_NMOS_GSD
- removed R30: 1k, Resistor_SMD:R_0402_1005Metric, symbol Device:R_Small
Connections:
- net PGOOD: no longer names the net of R25.2, U6.14 (P_GOOD)
Changed lines of the file:
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@@
   (junction (at 87.63 115.57) (diameter 0) (color 0 0 0 0)
   )
-  (junction (at 134.62 119.38) (diameter 0) (color 0 0 0 0)
-  )
   (junction (at 95.25 27.94) (diameter 0) (color 0 0 0 0)
   )
@@
   )
   (junction (at 86.36 27.94) (diameter 0) (color 0 0 0 0)
-  )
-  (junction (at 146.05 111.76) (diameter 0) (color 0 0 0 0)
   )
   (junction (at 124.46 49.53) (diameter 0) (color 0 0 0 0)
@@
     (stroke (width 0) (type default))
   )
-  (wire (pts (xy 146.05 114.3) (xy 146.05 111.76))
-    (stroke (width 0) (type default))
-  )
   (wire (pts (xy 74.93 60.96) (xy 74.93 63.5))
     (stroke (width 0) (type default))
@@
     (stroke (width 0) (type default))
   )
-  (wire (pts (xy 134.62 119.38) (xy 138.43 119.38))
-    (stroke (width 0) (type default))
-  )
   (wire (pts (xy 86.36 120.65) (xy 91.44 120.65))
     (stroke (width 0) (type default))
@@
     (stroke (width 0) (type default))
   )
-  (wire (pts (xy 132.08 119.38) (xy 134.62 119.38))
-    (stroke (width 0) (type default))
-  )
   (wire (pts (xy 100.33 115.57) (xy 109.22 115.57))
     (stroke (width 0) (type default))
@@
     (stroke (width 0) (type default))
   )
-  (wire (pts (xy 146.05 125.73) (xy 146.05 124.46))
-    (stroke (width 0) (type default))
-  )
   (wire (pts (xy 167.64 88.9) (xy 172.72 88.9))
     (stroke (width 0) (type default))
@@
   )
   (wire (pts (xy 58.42 66.04) (xy 63.5 66.04))
-    (stroke (width 0) (type default))
-  )
-  (wire (pts (xy 134.62 120.65) (xy 134.62 119.38))
     (stroke (width 0) (type default))
   )
@@
     )
   )
-  (hierarchical_label "BUCKC_EN" (shape input) (at 132.08 119.38 180) (fields_autoplaced)
-    (effects (font (size 1.27 1.27)) (justify right))
-  )
-  (hierarchical_label "PGOOD" (shape output) (at 72.39 83.82 180) (fields_autoplaced)
-    (effects (font (size 1.27 1.27)) (justify right))
-  )
   (symbol (lib_id "power:GNDA") (at 57.15 92.71 0) (unit 1)
     (in_bom yes) (on_board yes) (dnp no) (fields_autoplaced)
@@
     )
   )
-  (symbol (lib_id "power:GND") (at 134.62 125.73 0) (unit 1)
-    (in_bom yes) (on_board yes) (dnp no) (fields_autoplaced)
-    (property "Reference" "#PWR073" (at 134.62 132.08 0)
-      (effects (font (size 1.27 1.27)) hide)
-    )
-    (property "Value" "GND" (at 136.525 127.4338 0)
-      (effects (font (size 1.27 1.27)) (justify left))
-    )
-    (property "Footprint" "" (at 134.62 125.73 0)
-      (effects (font (size 1.27 1.27)) hide)
-    )
-    (property "Datasheet" "" (at 134.62 125.73 0)
-      (effects (font (size 1.27 1.27)) hide)
-    )
-    (pin "1")
-    (instances
-      (project "Ricardo-Stark"
-        (path "/7db990e4-92e1-4f99-b4d2-435bbec1ba83/6c17bf58-bab3-4fa6-ad33-cca9e388d73c"
-          (reference "#PWR073") (unit 1)
-        )
-      )
-    )
-  )
   (symbol (lib_id "power:GND") (at 121.92 83.82 0) (unit 1)
     (in_bom yes) (on_board yes) (dnp no) (fields_autoplaced)
@@
     )
   )
-  (symbol (lib_id "Device:R_Small") (at 134.62 123.19 180) (unit 1)
-    (in_bom yes) (on_board yes) (dnp no)
-    (property "Reference" "R30" (at 130.81 121.92 0)
-      (effects (font (size 1.27 1.27)))
-    )
-    (property "Value" "1k" (at 130.81 124.4569 0)
-      (effects (font (size 1.27 1.27)))
-    )
-    (property "Footprint" "Resistor_SMD:R_0402_1005Metric" (at 134.62 123.19 0)
-      (effects (font (size 1.27 1.27)) hide)
-    )
-    (property "Datasheet" "~" (at 134.62 123.19 0)
-      (effects (font (size 1.27 1.27)) hide)
-    )
-    (pin "1")
-    (pin "2")
-    (instances
-      (project "Ricardo-Stark"
-        (path "/7db990e4-92e1-4f99-b4d2-435bbec1ba83/6c17bf58-bab3-4fa6-ad33-cca9e388d73c"
-          (reference "R30") (unit 1)
-        )
-      )
-    )
-  )
   (symbol (lib_id "Device:C_Small") (at 163.322 68.072 0) (unit 1)
     (in_bom yes) (on_board yes) (dnp no) (fields_autoplaced)
@@
         (path "/7db990e4-92e1-4f99-b4d2-435bbec1ba83/6c17bf58-bab3-4fa6-ad33-cca9e388d73c"
           (reference "L4") (unit 1)
-        )
-      )
-    )
-  )
-  (symbol (lib_id "power:GND") (at 146.05 125.73 0) (unit 1)
-    (in_bom yes) (on_board yes) (dnp no) (fields_autoplaced)
-    (property "Reference" "#PWR075" (at 146.05 132.08 0)
-      (effects (font (size 1.27 1.27)) hide)
-    )
-    (property "Value" "GND" (at 147.955 127.4338 0)
-      (effects (font (size 1.27 1.27)) (justify left))
-    )
-    (property "Footprint" "" (at 146.05 125.73 0)
-      (effects (font (size 1.27 1.27)) hide)
-    )
-    (property "Datasheet" "" (at 146.05 125.73 0)
-      (effects (font (size 1.27 1.27)) hide)
-    )
-    (pin "1")
-    (instances
-      (project "Ricardo-Stark"
-        (path "/7db990e4-92e1-4f99-b4d2-435bbec1ba83/6c17bf58-bab3-4fa6-ad33-cca9e388d73c"
-          (reference "#PWR075") (unit 1)
         )
       )
@@
         )
       )
-    )
-  )
-  (symbol (lib_id "Device:Q_NMOS_GSD") (at 143.51 119.38 0) (unit 1)
-    (in_bom yes) (on_board yes) (dnp no)
-    (property "Reference" "Q1" (at 149.86 116.84 0)
-      (effects (font (size 1.27 1.27)) (justify left))
-    )
-    (property "Value" "SSM3K15AMFV,L3F" (at 149.86 120.015 0)
-      (effects (font (size 1.27 1.27)) (justify left))
-    )
-    (property "Footprint" "Package_TO_SOT_SMD:SOT-723" (at 148.59 116.84 0)
-      (effects (font (size 1.27 1.27)) hide)
-    )
-    (property "Datasheet" "~" (at 143.51 119.38 0)
-      (effects (font (size 1.27 1.27)) hide)
-    )
-    (pin "1")
-    (pin "2")
-    (pin "3")
-    (instances
-      (project "Ricardo-Stark"
-        (path "/7db990e4-92e1-4f99-b4d2-435bbec1ba83/6c17bf58-bab3-4fa6-ad33-cca9e388d73c"
-          (reference "Q1") (unit 1)
-        )
-      )

Commit message: commit
Parts:
- C29: value 68uF -> 470uF; footprint Capacitor_SMD:C_1206_3216Metric -> Capacitor_SMD:CP_Elec_6.3x7.7
- C31, C33: value 220uF -> 10uF; footprint Capacitor_SMD:C_1206_3216Metric -> Capacitor_SMD:C_0805_2012Metric
Connections:
- net +6V: now also C29.2; no longer C29.1
- net GND: now also C29.1; no longer C29.2

Commit message: commit
Connections:
- net +6V: now also C29.1; no longer C29.2
- net GND: now also C29.2; no longer C29.1
Other:
- moved on the sheet: C29
Changed lines of the file:
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@@
 	(symbol
 		(lib_id "Device:C_Small")
-		(at 92.456 118.11 180)
+		(at 92.456 118.11 0)
 		(unit 1)
 		(exclude_from_sim no)
@@
 		(fields_autoplaced yes)
 		(property "Reference" "C29"
-			(at 94.996 116.8336 0)
+			(at 95.25 116.8462 0)
 			(effects
 				(font
 					(size 1.27 1.27)
 				)
-				(justify right)
+				(justify left)
 			)
 		)
 		(property "Value" "470uF"
-			(at 94.996 119.3736 0)
+			(at 95.25 119.3862 0)
 			(effects
 				(font
 					(size 1.27 1.27)
 				)
-				(justify right)
+				(justify left)
 			)
 		)

Commit message: commit
Parts:
- removed C33: 10uF, Capacitor_SMD:C_0805_2012Metric, symbol Device:C_Small
- L4: footprint iclr:IND_SRP6540-390M -> Inductor_SMD:ETQP5M6M_YLC
Changed lines of the file:
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@@
-	)
-	(junction
-		(at 86.868 115.57)
-		(diameter 0)
-		(color 0 0 0 0)
-	)
-	(junction
-		(at 86.868 120.65)
-		(diameter 0)
-		(color 0 0 0 0)
 	)
 	(junction
@@
 		)
 	)
-	(wire
-		(pts
-			(xy 82.296 120.65) (xy 86.868 120.65)
-		)
-		(stroke
-			(width 0)
-			(type default)
-		)
-	)
 	(polyline
 		(pts
@@
 		(pts
 			(xy 62.23 20.32) (xy 64.77 20.32)
-		)
-		(stroke
-			(width 0)
-			(type default)
-		)
-	)
-	(wire
-		(pts
-			(xy 82.296 115.57) (xy 86.868 115.57)
 		)
 		(stroke
@@
 	)
 	(symbol
-		(lib_id "Device:C_Small")
-		(at 82.296 118.11 0)
-		(unit 1)
-		(exclude_from_sim no)
-		(in_bom yes)
-		(on_board yes)
-		(dnp no)
-		(property "Reference" "C33"
-			(at 80.518 114.046 0)
-			(effects
-				(font
-					(size 1.27 1.27)
-				)
-				(justify left)
-			)
-		)
-		(property "Value" "10uF"
-			(at 75.184 118.11 0)
-			(effects
-				(font
-					(size 1.27 1.27)
-				)
-				(justify left)
-			)
-		)
-		(property "Footprint" "Capacitor_SMD:C_0805_2012Metric"
-			(at 82.296 118.11 0)
-			(effects
-				(font
-					(size 1.27 1.27)
-				)
-				(hide yes)
-			)
-		)
-		(property "Datasheet" "~"
-			(at 82.296 118.11 0)
-			(effects
-				(font
-					(size 1.27 1.27)
-				)
-				(hide yes)
-			)
-		)
-		(property "Description" ""
-			(at 82.296 118.11 0)
-			(effects
-				(font
-					(size 1.27 1.27)
-				)
-				(hide yes)
-			)
-		)
-		(pin "1"
-		)
-		(pin "2"
-		)
-		(instances
-			(project "Ricardo-Stark"
-				(path "/7db990e4-92e1-4f99-b4d2-435bbec1ba83/6c17bf58-bab3-4fa6-ad33-cca9e388d73c"
-					(reference "C33")
-					(unit 1)
-				)
-			)
-		)
-	)
-	(symbol
 		(lib_id "power:+6V")
 		(at 114.046 115.57 0)
@@
 			)
 		)
-		(property "Footprint" "iclr:IND_SRP6540-390M"
+		(property "Footprint" "Inductor_SMD:ETQP5M6M_YLC"
 			(at 67.31 66.04 0)
 			(effects

Commit message: more changes
Parts:
- removed C28: 47uF, Capacitor_SMD:C_1206_3216Metric, symbol Device:C_Small
- removed C31: 10uF, Capacitor_SMD:C_0805_2012Metric, symbol Device:C_Small
Changed lines of the file:
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@@
 	(paper "A4")
-	(junction
-		(at 77.47 33.02)
-		(diameter 0)
-		(color 0 0 0 0)
-	)
 	(junction
 		(at 74.93 52.07)
@@
 	)
 	(junction
-		(at 77.47 27.94)
-		(diameter 0)
-		(color 0 0 0 0)
-	)
-	(junction
 		(at 95.25 27.94)
 		(diameter 0)
@@
 	)
 	(junction
-		(at 92.456 120.65)
-		(diameter 0)
-		(color 0 0 0 0)
-	)
-	(junction
 		(at 68.58 27.94)
 		(diameter 0)
@@
 	(wire
 		(pts
-			(xy 68.58 27.94) (xy 77.47 27.94)
+			(xy 68.58 27.94) (xy 82.55 27.94)
 		)
 		(stroke
@@
 	(wire
 		(pts
-			(xy 86.868 115.57) (xy 92.456 115.57)
-		)
-		(stroke
-			(width 0)
-			(type default)
-		)
-	)
-	(wire
-		(pts
 			(xy 57.15 86.36) (xy 57.15 87.63)
 		)
@@
 	(wire
 		(pts
-			(xy 68.58 33.02) (xy 77.47 33.02)
+			(xy 68.58 33.02) (xy 81.28 33.02)
 		)
 		(stroke
@@
 	(wire
 		(pts
-			(xy 77.47 27.94) (xy 82.55 27.94)
-		)
-		(stroke
-			(width 0)
-			(type default)
-		)
-	)
-	(wire
-		(pts
 			(xy 92.456 115.57) (xy 114.046 115.57)
 		)
@@
 	(wire
 		(pts
-			(xy 77.47 33.02) (xy 81.28 33.02)
-		)
-		(stroke
-			(width 0)
-			(type default)
-		)
-	)
-	(wire
-		(pts
 			(xy 58.42 86.36) (xy 57.15 86.36)
 		)
@@
 		(pts
 			(xy 74.93 66.04) (xy 74.93 68.58)
-		)
-		(stroke
-			(width 0)
-			(type default)
-		)
-	)
-	(wire
-		(pts
-			(xy 86.868 120.65) (xy 92.456 120.65)
 		)
 		(stroke
@@
 	(symbol
 		(lib_id "Device:C_Small")
-		(at 77.47 30.48 0)
-		(unit 1)
-		(exclude_from_sim no)
-		(in_bom yes)
-		(on_board yes)
-		(dnp no)
-		(fields_autoplaced yes)
-		(property "Reference" "C28"
-			(at 80.01 29.2163 0)
-			(effects
-				(font
-					(size 1.27 1.27)
-				)
-				(justify left)
-			)
-		)
-		(property "Value" "47uF"
-			(at 80.01 31.7563 0)
-			(effects
-				(font
-					(size 1.27 1.27)
-				)
-				(justify left)
-			)
-		)
-		(property "Footprint" "Capacitor_SMD:C_1206_3216Metric"
-			(at 77.47 30.48 0)
-			(effects
-				(font
-					(size 1.27 1.27)
-				)
-				(hide yes)
-			)
-		)
-		(property "Datasheet" "~"
-			(at 77.47 30.48 0)
-			(effects
-				(font
-					(size 1.27 1.27)
-				)
-				(hide yes)
-			)
-		)
-		(property "Description" ""
-			(at 77.47 30.48 0)
-			(effects
-				(font
-					(size 1.27 1.27)
-				)
-				(hide yes)
-			)
-		)
-		(pin "1"
-		)
-		(pin "2"
-		)
-		(instances
-			(project "Ricardo-Stark"
-				(path "/7db990e4-92e1-4f99-b4d2-435bbec1ba83/6c17bf58-bab3-4fa6-ad33-cca9e388d73c"
-					(reference "C28")
-					(unit 1)
-				)
-			)
-		)
-	)
-	(symbol
-		(lib_id "Device:C_Small")
 		(at 67.31 78.74 90)
 		(unit 1)
@@
 					(unit 1)
 				)
-			)
-		)
-	)
-	(symbol
-		(lib_id "Device:C_Small")
-		(at 86.868 118.11 0)
-		(unit 1)
-		(exclude_from_sim no)
-		(in_bom yes)
-		(on_board yes)
-		(dnp no)
-		(property "Reference" "C31"
-			(at 85.344 113.792 0)
-			(effects
-				(font
-					(size 1.27 1.27)
-				)
-				(justify left)
-			)
-		)
-		(property "Value" "10uF"
-			(at 84.328 122.682 0)
-			(effects
-				(font
-					(size 1.27 1.27)
-				)
-				(justify left)
-			)
-		)
-		(property "Footprint" "Capacitor_SMD:C_0805_2012Metric"
-			(at 86.868 118.11 0)
-			(effects
-				(font
-					(size 1.27 1.27)
-				)
-				(hide yes)
-			)
-		)
-		(property "Datasheet" "~"
-			(at 86.868 118.11 0)
-			(effects
-				(font
-					(size 1.27 1.27)
-				)
-				(hide yes)
-			)
-		)
-		(property "Description" ""
-			(at 86.868 118.11 0)
-			(effects
-				(font
-					(size 1.27 1.27)
-				)
-				(hide yes)
-			)
-		)
-		(pin "1"
-		)
-		(pin "2"
-		)
-		(instances
-			(project "Ricardo-Stark"
-				(path "/7db990e4-92e1-4f99-b4d2-435bbec1ba83/6c17bf58-bab3-4fa6-ad33-cca9e388d73c"
-					(reference "C31")
-					(unit 1)
-				)
