File: power.kicad_sch (KiCad schematic)
At the start: 20 parts, among them U3 LM66200DRLR, U4 MAX77827AEFD+T, U5 SC4215

Commit message: Completed schematics
Parts:
- renumbered C20 to C17, C21 to C18, C22 to C19, C23 to C20, C24 to C21, C25 to C22, C26 to C23, C27 to C24, R14 to R15, R15 to R16, R16 to R17, R17 to R18, TP4 to TP5, TP5 to TP6, TP6 to TP7

Commit message: More Based
Parts:
- renumbered R15 to R21, R16 to R22, R17 to R23, R18 to R24

Commit message: more changes
Connections:
- net RBUS_uC_V: now also U3.3 (VIN1); no longer U3.6 (VIN2)
- net VBUS: now also U3.6 (VIN2); no longer U3.3 (VIN1)
Changed lines of the file:
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@@
 	(global_label "RBUS_uC_V"
 		(shape input)
-		(at 90.17 39.37 0)
+		(at 34.29 41.91 180)
 		(fields_autoplaced yes)
 		(effects
@@
 				(size 1.27 1.27)
 			)
-			(justify left)
+			(justify right)
 		)
 		(property "Intersheetrefs" "${INTERSHEET_REFS}"
-			(at 103.0171 39.4494 0)
-			(effects
-				(font
-					(size 1.27 1.27)
-				)
-				(justify left)
+			(at 21.4362 41.91 0)
+			(effects
+				(font
+					(size 1.27 1.27)
+				)
+				(justify right)
 				(hide yes)
 			)
@@
 	(symbol
 		(lib_id "power:VBUS")
-		(at 34.29 41.91 0)
+		(at 90.17 39.37 0)
 		(unit 1)
 		(exclude_from_sim no)
@@
 		(fields_autoplaced yes)
 		(property "Reference" "#PWR044"
-			(at 34.29 45.72 0)
+			(at 90.17 43.18 0)
 			(effects
 				(font
@@
 		)
 		(property "Value" "VBUS"
-			(at 34.29 38.3342 0)
+			(at 90.17 35.7942 0)
 			(effects
 				(font
@@
 		)
 		(property "Footprint" ""
-			(at 34.29 41.91 0)
+			(at 90.17 39.37 0)
 			(effects
 				(font
@@
 		)
 		(property "Datasheet" ""
-			(at 34.29 41.91 0)
+			(at 90.17 39.37 0)
 			(effects
 				(font
@@
 		)
 		(property "Description" ""
-			(at 34.29 41.91 0)
-			(effects
-				(font
+			(at 90.17 39.37 0)
+			(effects
+				(font
