File: Ricardo-Stark.kicad_sch (KiCad schematic)
At the start: 54 parts, among them J1 RBUS, U1 ESP32-S3, Y1 R940000171

Commit message: review 3 changes
Connections:
- net ADS_CS0: now also U1.41 (GPIO36); no longer U1.40 (GPIO35)
- net GPIO4: now also U1.44 (MTCK/JTAG/GPIO39); no longer U1.43 (GPIO38)
- net GPIO5: now also U1.48 (MTMS/JTAG/GPIO42); no longer U1.47 (MTDI/JTAG/GPIO41)
- net GPIO7: now also U1.47 (MTDI/JTAG/GPIO41); no longer U1.44 (MTCK/JTAG/GPIO39)
- net GPIO8: now also U1.42 (GPIO37); no longer U1.41 (GPIO36)
- net GPIO9: now also U1.43 (GPIO38); no longer U1.42 (GPIO37)
- new net DRDY: U1.40 (GPIO35)
- no-connect marks 15 -> 14
Other:
- sheet pressure_sensor ports: added DRDY; removed none
Changed lines of the file:
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@@
 		(at 135.89 80.01)
 	)
-	(no_connect
-		(at 69.85 125.73)
-	)
 	(wire
 		(pts
@@
 		)
 	)
+	(label "DRDY"
+		(at 135.89 100.33 0)
+		(fields_autoplaced yes)
+		(effects
+			(font
+				(size 1.27 1.27)
+			)
+			(justify left bottom)
+		)
+	)
 	(label "CAN+"
 		(at 115.57 185.42 0)
@@
 	)
 	(label "GPIO7"
-		(at 69.85 118.11 180)
+		(at 69.85 123.19 180)
 		(fields_autoplaced yes)
 		(effects
@@
 	)
 	(label "GPIO9"
-		(at 135.89 105.41 0)
+		(at 135.89 107.95 0)
 		(fields_autoplaced yes)
 		(effects
@@
 		)
 	)
+	(label "DRDY"
+		(at 182.88 84.074 180)
+		(fields_autoplaced yes)
+		(effects
+			(font
+				(size 1.27 1.27)
+			)
+			(justify right bottom)
+		)
+	)
 	(label "CAN_TX"
 		(at 14.732 33.274 0)
@@
 	)
 	(label "GPIO8"
-		(at 135.89 102.87 0)
+		(at 135.89 105.41 0)
 		(fields_autoplaced yes)
 		(effects
@@
 	)
 	(label "GPIO5"
-		(at 69.85 123.19 180)
+		(at 69.85 125.73 180)
 		(fields_autoplaced yes)
 		(effects
@@
 	)
 	(label "ADS_CS0"
-		(at 135.89 100.33 0)
+		(at 135.89 102.87 0)
 		(fields_autoplaced yes)
 		(effects
@@
 	)
 	(label "GPIO4"
-		(at 135.89 107.95 0)
+		(at 69.85 118.11 180)
 		(fields_autoplaced yes)
 		(effects
@@
 				(size 1.27 1.27)
 			)
-			(justify left bottom)
+			(justify right bottom)
 		)
 	)
@@
 			)
 		)
+		(pin "DRDY" bidirectional
+			(at 182.88 84.074 180)
+			(effects
+				(font
+					(size 1.27 1.27)
+				)
+				(justify left)
+			)
+		)

Commit message: Changed sd card holder
Connections:
- net SD1_CS: now also U1.11 (GPIO6/ADC1_CH5); no longer U1.14 (GPIO9/ADC1_CH8)
- net VSPI_MISO: now also U1.14 (GPIO9/ADC1_CH8); no longer U1.11 (GPIO6/ADC1_CH5)
- net VSPI_MOSI: now also U1.12 (GPIO7/ADC1_CH6); no longer U1.13 (GPIO8/ADC1_CH7)
- net VSPI_SCLK: now also U1.13 (GPIO8/ADC1_CH7); no longer U1.12 (GPIO7/ADC1_CH6)
- net GPIO4 renamed GPIO39
- net GPIO5 renamed GPIO42
- net GPIO6 renamed GPIO40
- net GPIO7 renamed GPIO41
- net GPIO8 renamed GPIO37
- net GPIO9 renamed GPIO38
Other:
- sheet actuators ports: added GPIO37, GPIO38, GPIO39, GPIO40, GPIO41, GPIO42; removed GPIO4, GPIO5, GPIO6, GPIO7, GPIO8, GPIO9
- sheet microSD ports: added SD_DET; removed SD1_DET
Changed lines of the file:
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@@
 	(wire
 		(pts
-			(xy 254.508 58.293) (xy 257.556 58.293)
+			(xy 254.508 58.42) (xy 257.556 58.42)
 		)
 		(stroke
@@
 	(wire
 		(pts
-			(xy 187.96 64.008) (xy 180.34 64.008)
+			(xy 187.96 64.008) (xy 177.546 64.008)
 		)
 		(stroke
@@
 		)
 	)
-	(label "GPIO7"
+	(label "GPIO38"
 		(at 187.96 53.848 180)
 		(fields_autoplaced yes)
@@
 		)
 	)
-	(label "GPIO6"
+	(label "GPIO37"
 		(at 187.96 51.562 180)
 		(fields_autoplaced yes)
@@
 		)
 	)
-	(label "GPIO7"
+	(label "GPIO41"
 		(at 69.85 123.19 180)
 		(fields_autoplaced yes)
@@
 	)
 	(label "VSPI_SCLK"
-		(at 69.85 87.63 180)
+		(at 69.85 90.17 180)
 		(fields_autoplaced yes)
 		(effects
@@
 	)
 	(label "SD1_CS"
-		(at 69.85 92.71 180)
+		(at 69.85 85.09 180)
 		(fields_autoplaced yes)
 		(effects
@@
 		)
 	)
-	(label "GPIO9"
+	(label "GPIO38"
 		(at 135.89 107.95 0)
 		(fields_autoplaced yes)
@@
 	)
 	(label "VSPI_MISO"
-		(at 69.85 85.09 180)
+		(at 69.85 92.71 180)
 		(fields_autoplaced yes)
 		(effects
@@
 		)
 	)
-	(label "GPIO8"
+	(label "GPIO37"
 		(at 135.89 105.41 0)
 		(fields_autoplaced yes)
@@
 	)
 	(label "SD1_DET"
-		(at 254.508 58.293 180)
+		(at 254.508 58.42 180)
 		(fields_autoplaced yes)
 		(effects
@@
 		)
 	)
-	(label "GPIO5"
+	(label "GPIO42"
 		(at 69.85 125.73 180)
 		(fields_autoplaced yes)
@@
 		)
 	)
-	(label "GPIO6"
+	(label "GPIO40"
 		(at 69.85 120.65 180)
 		(fields_autoplaced yes)
@@
 		)
 	)
-	(label "GPIO9"
+	(label "GPIO42"
 		(at 187.96 62.484 180)
 		(fields_autoplaced yes)
@@
 		)
 	)
-	(label "GPIO4"
+	(label "GPIO39"
 		(at 187.96 56.134 180)
 		(fields_autoplaced yes)
@@
 		)
 	)
-	(label "GPIO8"
+	(label "GPIO41"
 		(at 187.96 60.452 180)
 		(fields_autoplaced yes)
@@
 	)
 	(label "VSPI_MOSI"
-		(at 69.85 90.17 180)
+		(at 69.85 87.63 180)
 		(fields_autoplaced yes)
 		(effects
@@
 		)
 	)
-	(label "GPIO4"
+	(label "GPIO39"
 		(at 69.85 118.11 180)
 		(fields_autoplaced yes)
@@
 		)
 	)
-	(label "GPIO5"
+	(label "GPIO40"
 		(at 187.96 58.166 180)
 		(fields_autoplaced yes)
@@
 	(symbol
 		(lib_id "power:+5V")
-		(at 180.34 64.008 180)
+		(at 177.546 64.008 0)
 		(unit 1)
 		(exclude_from_sim no)
@@
 		(fields_autoplaced yes)
 		(property "Reference" "#PWR092"
-			(at 180.34 60.198 0)
+			(at 177.546 67.818 0)
 			(effects
 				(font
@@
 		)
 		(property "Value" "+5V"
-			(at 180.34 69.088 0)
+			(at 177.546 59.69 0)
 			(effects
 				(font
@@
 		)
 		(property "Footprint" ""
-			(at 180.34 64.008 0)
+			(at 177.546 64.008 0)
 			(effects
 				(font
@@
 		)
 		(property "Datasheet" ""
-			(at 180.34 64.008 0)
+			(at 177.546 64.008 0)
 			(effects
 				(font
@@
 		)
 		(property "Description" ""
-			(at 180.34 64.008 0)
+			(at 177.546 64.008 0)
 			(effects
 				(font
@@
 			)
 		)
-		(pin "GPIO6" input
-			(at 187.96 51.562 180)
+		(pin "5V" output
+			(at 187.96 64.008 180)
 			(effects
 				(font
@@
 			)
 		)
-		(pin "GPIO7" input
+		(pin "GPIO38" input
 			(at 187.96 53.848 180)
 			(effects
@@
 			)
 		)
-		(pin "GPIO4" input
-			(at 187.96 56.134 180)
+		(pin "GPIO37" input
+			(at 187.96 51.562 180)
 			(effects
 				(font
@@
 			)
 		)
-		(pin "GPIO5" input
-			(at 187.96 58.166 180)
+		(pin "GPIO41" input
+			(at 187.96 60.452 180)
 			(effects
 				(font
@@
 			)
 		)
-		(pin "GPIO8" input
-			(at 187.96 60.452 180)
+		(pin "GPIO39" input
+			(at 187.96 56.134 180)
 			(effects
 				(font
@@
 			)
 		)
-		(pin "GPIO9" input
-			(at 187.96 62.484 180)
+		(pin "GPIO40" input
+			(at 187.96 58.166 180)
 			(effects
 				(font
@@
 			)
 		)
-		(pin "5V" output
-			(at 187.96 64.008 180)
+		(pin "GPIO42" input
+			(at 187.96 62.484 180)
 			(effects
 				(font
@@
 			)
 		)
-		(pin "SD1_DET" input
-			(at 257.556 58.293 180)
-			(effects
-				(font
-					(size 1.27 1.27)
-				)
-				(justify left)
-			)
-		)
 		(pin "VSPI_SCLK" input
 			(at 257.556 54.483 180)
@@
 			(effects
 				(font
+					(size 1.27 1.27)
+				)
+				(justify left)
+			)
+		)
+		(pin "SD_DET" input
+			(at 257.556 58.42 180)
+			(effects
+				(font
