File: Hardware/Pyro.kicad_sch (KiCad schematic)
At the start: 36 parts, among them IC5 TPS259830ONRGER, J12 Conn_01x02_Male, Q2 BUK9M11-40EX, U10 SiC437BED-T1-GE3, U9 782-TCMT1109

Commit message: updated sensors and other stuff
Parts:
- removed C45: 4.7nF, Capacitor_SMD:C_0402_1005Metric, symbol Device:C_Small
- removed C46: 10nF, Capacitor_SMD:C_0402_1005Metric, symbol Device:C_Small
- removed D6: 954-S-102T, Diode_SMD:D_1206_3216Metric, symbol Device:D
- removed IC5: TPS259830ONRGER, iclr:TPS259830ONRGER, symbol iclr:TPS259830ONRGER
- removed R108: 1M, Capacitor_SMD:C_0402_1005Metric, symbol Device:R_Small
- removed R109: 732k, Capacitor_SMD:C_0402_1005Metric, symbol Device:R_Small
- removed R110: 73.2k, Capacitor_SMD:C_0402_1005Metric, symbol Device:R_Small
- removed R111: 300, Capacitor_SMD:C_0402_1005Metric, symbol Device:R_Small
- removed R112: 681, Capacitor_SMD:C_0402_1005Metric, symbol Device:R_Small
- removed R113: 100k, Capacitor_SMD:C_0402_1005Metric, symbol Device:R_Small
- added D9: S-102T, iclr:SODFL3516X70N, symbol Device:D_Current-regulator
- J12: footprint TerminalBlock_Phoenix:TerminalBlock_Phoenix_PT-1,5-2-3.5-H_1x02_P3.50mm_Horizontal -> Connector_Molex:Molex_Nano-Fit_105313-xx02_1x02_P2.50mm_Horizontal
Connections:
- net GND: now also D9.1 (K)
- net PyroV: now also J12.2 (Pin_2); no longer J12.1 (Pin_1)
- net VDD: no longer C73.2, R81.1
- net at D3.1 (A), D3.2 (A), U9.1: now also J12.1 (Pin_1); no longer J12.2 (Pin_2)
- net at U9.2: now also D9.2 (A)
- new net: C73.2, R81.1
- no-connect marks 5 -> 3
Other:
- note removed: "SPM10065VT-3R3M-D"
- note removed: "dvdt pin left floating for fastest turn on time"
- moved on the sheet: C27, C40, C73, C74, C75, C76, C83, L7, R42, R43, R81, R82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
