File: Hardware/Fuzzzze.kicad_sch (KiCad schematic)
At the start: 22 parts, among them Q1 BSZ025N04LS, Q4 BSZ025N04LS, U11 LM74810, U12 INA219AxDCN

Commit message: Routed Switch and Servo driver subsystems
Parts:
- removed C45, C71, C72, C77: 0.1uF, Capacitor_SMD:C_0402_1005Metric, symbol Device:C_Small
- removed C46: 1uF, Capacitor_SMD:C_0402_1005Metric, symbol Device:C_Small
- removed C47: 0.1uF, Capacitor_SMD:C_0603_1608Metric, symbol Device:C_Small
- removed D8: P6SMBJ28CA, Diode_SMD:D_SMA, symbol Device:D_TVS_Small_Filled
- removed Q1, Q4: BSZ025N04LS, iclr:BSZ025N04LS, symbol iclr:BSZ025N04LS
- removed R108, R94: 10, Resistor_SMD:R_0402_1005Metric, symbol Device:R_Small
- removed R109, R110: 3.3k, Resistor_SMD:R_0402_1005Metric, symbol Device:R_Small
- removed R44: 10k, Resistor_SMD:R_0402_1005Metric, symbol Device:R_Small
- removed R80: 100k, Resistor_SMD:R_0402_1005Metric, symbol Device:R_Small
- removed R85: 5.1k, Resistor_SMD:R_0402_1005Metric, symbol Device:R_Small
- removed R89: 4.22k, Resistor_SMD:R_0402_1005Metric, symbol Device:R_Small
- removed R93: 2m, Resistor_SMD:R_2512_6332Metric_Pad1.40x3.35mm_HandSolder, symbol Device:R
- removed TP10, TP9: TestPoint, TestPoint:TestPoint_Pad_D1.0mm, symbol Connector:TestPoint
- removed U11: LM74810, iclr:SON50P300X300X80-13N-D, symbol iclr:LM74810QDRRRQ1
- removed U12: INA219AxDCN, Package_TO_SOT_SMD:SOT-23-8, symbol Sensor_Energy:INA219AxDCN
Connections:
- no-connect marks 1 -> 0
Other:
- note removed: "Batt Mon - 3.0V out @ 35V in Overvoltage cutoff - 32V Check sizing script"
