File: Hardware/Ricardo-Stark.kicad_pcb (KiCad board)
At the start: 4 copper layers, 124 x 56 mm, 337 parts, among them IC1 TPS61089RNRR, IC2 AP2205-W5-7, IC3 AP2205-W5-7, IC4 TPS61089RNRR, J1 RBUS, J10 1053131104, J11 Conn_01x08_Socket, J12 Conn_01x02_Male, J13 1053131104, J14 Conn_01x02_Male, J15 Conn_01x02_Male, J16 Conn_01x07_Socket, J17 ServoCH1, J18 ServoCH2, J2 USB_C_Receptacle_USB2.0, J3 ST1W008S4TR2000, J5 Conn_01x03_Socket, J6 1053131104, J7 1053131104, J8 1053131104, J9 1053131104, Q7 BSZ025N04LS, Q8 BSZ025N04LS, Q9 BSZ025N04LS, U1 ESP32-S3, U10 SiC438BED-T1-GE3, U11 782-TCMT1109, U12 INA219AxDCN, U13 MAX31856, U14 PCA9534RGVR, U15 782-TCMT1109, U2 SN65HVD230, U3 LM66200DRLR, U4 MAX77827AEFD+T, U5 SC4215, U6 SiC437BED-T1-GE3, U7 ADS131M06IPBS, U8 PCA9685BS, U9 782-TCMT1109, Y1 R940000171

Commit message: quick changes before silwood
Parts:
- moved JP12 8.49 mm to (119.6, 99.1), turned to 0 degrees
- moved JP17 6.67 mm to (139.5, 111.2), turned to 90 degrees
- moved JP33 6.60 mm to (182.9, 106.5), turned to 90 degrees
- moved JP10 6.58 mm to (119.5, 112.8), turned to 0 degrees
- moved JP28 6.56 mm to (168.9, 111.2), turned to 90 degrees
- moved JP23 6.54 mm to (154.2, 111.2), turned to 90 degrees
- moved L5 1.82 mm to (129.6, 78.0)
- moved C57 1.60 mm to (133.2, 72.1)
- moved L6 1.59 mm to (140.4, 68.1)
- moved C70 1.47 mm to (136.9, 74.0)
- moved R12 1.13 mm to (137.9, 77.3)
- moved R68 0.91 mm to (140.0, 76.2)
- moved R61 0.89 mm to (130.4, 70.0)
- moved R62 0.89 mm to (130.4, 71.0)
- moved R69 0.88 mm to (140.0, 75.2)
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Routing:
- net GND: track 404.9 -> 391.2 mm, vias 502 -> 548
- net +5V: track 146.1 -> 135.6 mm
- net +12V: track 124.5 -> 119.6 mm
- net Net-(IC1-BOOT): track 2.94 -> 0.00 mm
- net Net-(IC4-COMP): track 0.00 -> 2.42 mm
- net Net-(IC1-COMP): track 0.00 -> 2.16 mm
- net Net-(JP12-C): track 5.13 -> 2.99 mm
- net Net-(IC1-VCC): track 3.76 -> 2.41 mm
- net /SDA: track 143.8 -> 142.5 mm
- net Net-(JP28-C): track 5.94 -> 4.92 mm
- net Net-(IC4-VCC): track 3.18 -> 2.20 mm
- net /Boosts/LDO12V_IN: track 9.92 -> 8.96 mm
- net Net-(3V3LED8-A): track 3.79 -> 2.86 mm
- net Net-(JP33-C): track 4.63 -> 3.92 mm
- net +3.3V: track 52.9 -> 53.0 mm, vias 36 -> 38
- added copper zone on F.Cu, net Net-(IC1-BOOT)
- removed copper zone on F.Cu, net Net-(IC1-COMP)
- removed copper zone on F.Cu, net Net-(IC4-COMP)
