File: Hardware/Ricardo-Stark.kicad_pcb (KiCad board)
At the start: 4 copper layers, 124 x 56 mm, 337 parts, among them J1001 Conn_01x07_Socket, J1002 ST1W008S4TR2000, J101 Conn_01x02_Male, J102 Conn_01x02_Male, J103 RBUS, J104 Conn_01x03_Socket, J105 Conn_01x08_Socket, J501 USB_C_Receptacle_USB2.0, J701 Thermocouple, J702 1053131104, J703 1053131104, J704 1053131104, J705 1053131104, J706 1053131104, J707 1053131104, J801 ServoCH1, J802 ServoCH2, J901 Conn_01x02_Male, J902 Conn_01x02_Male, J903 Conn_01x02_Male, Q901 BSZ025N04LS, Q902 BSZ025N04LS, Q903 BSZ025N04LS, U101 ESP32-S3, U102 PCA9534RGVR, U201 LM66200DRLR, U202 MAX77827AEFD+T, U203 SC4215ASTRT, U301 SiC437BED-T1-GE3, U401 TPS61089RNRR, U402 AP2205-W5-7, U403 AP2205-W5-7, U404 TPS61089RNRR, U601 SN65HVD230, U701 ADS131M06IPBS, U702 MAX31856, U801 PCA9685BS, U901 SiC438BED-T1-GE3, U902 782-TCMT1109, U903 782-TCMT1109, U904 INA219AxDCN, U905 782-TCMT1109, Y101 40MHz±10ppm

Commit message: changed fp
Parts:
- D103, D104, D105, D502: footprint Resistor_SMD:R_0402_1005Metric -> LED_SMD:LED_0402_1005Metric
- U301: value SiC437BED-T1-GE3 -> SIC437AED-T1-GE3
- U901: value SiC438BED-T1-GE3 -> SIC437AED-T1-GE3
- U902, U903, U905: value 782-TCMT1109 -> TCMT1109; footprint iclr:TCMT1109-4N -> Package_SO:SOP-4_4.4x2.6mm_P1.27mm
